Commit message: Fixed urdf file

File: urdf/basic_pig.urdf.xacro (robot description, xacro)
@@ -2,7 +2,10 @@
 <robot name="basic_pig"
     xmlns:xacro="http://www.ros.org/wiki/xacro">
+    <!-- Standard Params -->
+    <xacro:property name="pi" value="3.1415" />
     <!-- Degree-to-radian conversions -->
     <xacro:property name="degrees_45" value="0.785398163"/>
     <xacro:property name="degrees_90" value="1.57079633"/>
+    <xacro:property name="degrees_180" value="3.14159265"/>
     <!-- Inertia Generator -->
     <xacro:macro name="default_inertial" params="mass">
@@ -12,18 +15,25 @@
         </inertial>
     </xacro:macro>
+    <xacro:property name="axle_eff_limit" value="100"/>
+    <xacro:property name="axle_vel_limit" value="39.02"/>
+    <!-- Servo_stall_torque of the direction axis in Nm. servo_no_load_speed is
+       measured in rad/s. -->
+    <xacro:property name="servo_stall_torque" value="100"/>
+    <xacro:property name="servo_no_load_speed" value="100"/>
     <!-- Basic Geometry of Body -->
     <xacro:property name="body_length" value="1.91" />
     <xacro:property name="body_width" value="0.680618" />
     <xacro:property name="body_height" value="1.065022" />
-    <xacro:property name="body_mass" value="41" />
+    <xacro:property name="body_mass" value="40"/>
+    <!-- The Ackerman Steering Hub -->
+    <xacro:property name="ackerman_joint_diameter" value="0.09" />
+    <xacro:property name="ackerman_joint_width" value="0.09" />
     <!-- Front Wheel Properties -->
     <xacro:property name="front_wheel_width" value=".254" />
     <xacro:property name="front_wheel_diameter" value="0.605" />
-    <xacro:property name="front_wheel_mass" value="10" />
     <!-- Rear Wheel Properties -->
     <xacro:property name="rear_wheel_width" value="0.2794" />
     <xacro:property name="rear_wheel_diameter" value="0.635" />
-    <xacro:property name="rear_wheel_mass" value="12" />
-    <!-- Main Body -->
+    <!-- Main Body of Little Pig -->
     <link name="base_link">
         <visual>
@@ -31,7 +41,7 @@
                 <box size="${body_length} ${body_width} ${body_height}"/>
             </geometry>
+            <material name="blue" />
         </visual>
         <collision>
-            <origin xyz="0.0 0.0 0.0" rpy="0.0 0.0 0.0"/>
             <geometry>
                 <box size="${body_length} ${body_width} ${body_height}"/>
@@ -40,8 +50,172 @@
         <xacro:default_inertial mass="${body_mass}" />
     </link>
+    <!-- Gazebo Interface -->
+    <gazebo reference="base_link">
+        <material>Gazebo/Blue</material>
+    </gazebo>
+    <!-- Ackerman Steering Macro -->
+    <xacro:macro name="ackerman_steering" params="prefix reflect">
+        <!-- The Link -->
+        <link name="${prefix}_ackerman_link">
+            <visual>
+                <origin xyz="0.0 0.0 0.0" rpy="${pi/2} 0.0 0.0"/>
+                <geometry>
+                    <cylinder radius="${ackerman_joint_diameter/2}" length="${ackerman_joint_width}"/>
+                </geometry>
+                <material name="black" />
+            </visual>
+            <collision>
+                <origin xyz="0.0 0.0 0.0" rpy="${pi/2} 0.0 0.0"/>
+                <geometry>
+                    <cylinder radius="${ackerman_joint_diameter/2}" length="${ackerman_joint_width}"/>
+                </geometry>
+            </collision>
+            <xacro:default_inertial mass="2"/>
+        </link>
+        <!-- The Joint -->
+        <joint name="base_link_${prefix}_ackerman_link" type="revolute">
+            <axis xyz="0.0 0.0 1.0" rpy="0.0 0.0 0.0"/>
+            <parent link="base_link"/>
+            <child link="${prefix}_ackerman_link"/>
+            <origin xyz="${body_length / 2.5} ${((ackerman_joint_width/2) + (body_width/2)) * reflect} -${(body_height / 2.25) + (ackerman_joint_diameter / 2)}" rpy="0.0 0.0 0.0"/>
+            <limit lower="${-degrees_45}" upper="${degrees_45}" effort="${servo_stall_torque}" velocity="${servo_no_load_speed}"/>
+        </joint>
+        <!-- Gazebo Interface -->
+        <gazebo reference="${prefix}_ackerman_link">
+            <mu1 value="1.0"/>
+            <mu2 value="1.0"/>
+            <kp value="10000000.0" />
+            <kd value="1.0" />
+            <fdir1 value="1 0 0"/>
+            <material>Gazebo/Black</material>
+        </gazebo>
+        <!-- The Transmission -->
+        <transmission name="base_link_${prefix}_ackerman_link_trans">
+            <type>transmission_interface/SimpleTransmission</type>
+            <joint name="base_link_${prefix}_ackerman_link">
+                <hardwareInterface>hardware_interface/EffortJointInterface</hardwareInterface>
+            </joint>
+            <actuator name="base_link_${prefix}_ackerman_link_motor">
+                <hardwareInterface>hardware_interface/EffortJointInterface</hardwareInterface>
+                <mechanicalReduction>1</mechanicalReduction>
+            </actuator>
+        </transmission>
+    </xacro:macro>
+    <!-- Front Wheel Macro -->
+    <xacro:macro name="front_wheel" params="prefix suffix reflect">
+        <!-- The Link -->
+        <link name="front_${suffix}_wheel">
+            <visual>
+                <origin xyz="0.0 ${(front_wheel_width/2) * reflect} 0.0" rpy="${pi/2} 0.0 0.0"/>
+                <geometry>
+                    <cylinder radius="${front_wheel_diameter/2}" length="${front_wheel_width}"/>
+                </geometry>
+                <material name="black" />
+            </visual>
+            <collision>
+                <origin xyz="0.0 0.0 0.0" rpy="${pi/2} 0.0 0.0"/>
+                <geometry>
+                    <cylinder radius="${front_wheel_diameter/2}" length="${front_wheel_width}"/>
+                </geometry>
+            </collision>
+            <inertial>
+                <origin xyz="0.0 0.0 0.0" rpy="0.0 0.0 0.0"/>
+                <mass value="20.995"/>
+                <inertia ixx="0.996" ixy="0.0" ixz="0.0" iyy="0.612" iyz="0.0" izz="0.612"/>
+            </inertial>
+        </link>
+        <!-- The Joint -->
+        <joint name="${prefix}_ackerman_link_front_${suffix}_wheel" type="continuous">
+            <axis xyz="0.0 1.0 0.0"/>
+            <parent link="${prefix}_ackerman_link"/>
+            <child link="front_${suffix}_wheel"/>
+            <origin xyz="0.0 0.0 0.0" rpy="0.0 0.0 0.0"/>
+            <limit effort="${axle_eff_limit}" velocity="${axle_vel_limit}"/>
+        </joint>
+        <!-- Gazebo Interface -->
+        <gazebo reference="front_${suffix}_wheel">
+            <mu1 value="1.0"/>
+            <mu2 value="1.0"/>
+            <kp value="10000000.0" />
+            <kd value="1.0" />
+            <fdir1 value="0 0 1"/>
+            <material>Gazebo/Black</material>
+        </gazebo>
+        <!-- The Transmission -->
+        <transmission name="${prefix}_ackerman_link_front_${suffix}_wheel_trans">
+            <type>transmission_interface/SimpleTransmission</type>
+            <joint name="${prefix}_ackerman_link_front_${suffix}_wheel">
+                <hardwareInterface>hardware_interface/VelocityJointInterface</hardwareInterface>
+            </joint>
+            <actuator name="${prefix}_ackerman_link_front_${suffix}_wheel_motor">
+                <hardwareInterface>hardware_interface/VelocityJointInterface</hardwareInterface>
+                <mechanicalReduction>1</mechanicalReduction>
+            </actuator>
+        </transmission>
+    </xacro:macro>
+    <!-- Back Wheel Macro -->
+    <xacro:macro name="rear_wheel" params="suffix reflect">
+        <!-- The Link -->
+        <link name="rear_${suffix}_wheel">
+            <visual>
+                <origin xyz="0.0 ${(rear_wheel_width / 2) * reflect} 0.0" rpy="${pi/2} 0.0 0.0"/>
+                <geometry>
+                    <cylinder radius="${rear_wheel_diameter/2}" length="${rear_wheel_width}"/>
+                </geometry>
+                <material name="black" />
+            </visual>
+            <collision>
+                <origin xyz="0.0 0.0 0.0" rpy="${pi/2} 0.0 0.0"/>
+                <geometry>
+                    <cylinder radius="${rear_wheel_diameter/2}" length="${rear_wheel_width}"/>
+                </geometry>
+            </collision>
+            <inertial>
+                <origin xyz="0.0 0.0 0.0" rpy="0.0 0.0 0.0"/>
+                <mass value="20.995"/>
+                <inertia ixx="0.996" ixy="0.0" ixz="0.0" iyy="0.612" iyz="0.0" izz="0.612"/>
+            </inertial>
+        </link>
+        <!-- The Joint -->
+        <joint name="base_to_rear_${suffix}_wheel" type="continuous">
+            <axis xyz="0.0 1.0 0.0"/>
+            <parent link="base_link"/>
+            <child link="rear_${suffix}_wheel"/>
+            <origin xyz="-${body_length / 2.5} ${(body_width /2) * reflect} -${(body_height / 5) + (rear_wheel_diameter / 2)}" rpy="0.0 0.0 0.0"/>
+        </joint>
+        <!-- Gazebo Interface -->
+        <gazebo reference="rear_${suffix}_wheel">
+            <!-- <mu1 value="1.0"/>
+            <mu2 value="1.0"/>
+            <kp value="10000000.0" />
+            <kd value="1.0" />
+            <fdir1 value="1 0 0"/> -->
+            <material>Gazebo/Black</material>
+        </gazebo>
+        <!-- The Transmission -->
+        <!-- <transmission name="base_to_rear_${suffix}_wheel_trans">
+            <type>transmission_interface/SimpleTransmission</type>
+            <joint name="base_to_rear_${suffix}_wheel">
+                <hardwareInterface>hardware_interface/VelocityJointInterface</hardwareInterface>
+            </joint>
+            <actuator name="base_to_rear_${suffix}_wheel_motor">
+                <hardwareInterface>hardware_interface/VelocityJointInterface</hardwareInterface>
+                <mechanicalReduction>1</mechanicalReduction>
+            </actuator>
+        </transmission> -->
+    </xacro:macro>
+    <!-- Call the ackermans in for left/right -->
+    <xacro:ackerman_steering prefix="left" reflect="1" />
+    <xacro:ackerman_steering prefix="right" reflect="-1" />
+    <!-- Call the front wheels in left/right -->
+    <xacro:front_wheel prefix="left" suffix="left" reflect="1" />
+    <xacro:front_wheel prefix="right" suffix="right" reflect="-1" />
+    <!-- Call the rear wheels in left/right-->
+    <xacro:rear_wheel suffix="left" reflect="1" />
+    <xacro:rear_wheel suffix="right" reflect="-1" />
     <!-- Gazebo plugin for ROS Control -->
     <gazebo>
         <plugin name="gazebo_ros_control" filename="libgazebo_ros_control.so">
-            <robotNamespace>/basic_pig</robotNamespace>
+            <robotNamespace>/basic_geometry_pig</robotNamespace>
         </plugin>
     </gazebo>

Commit message: minor update to base link

File: urdf/basic_pig.urdf.xacro (robot description, xacro)
@@ -54,4 +54,8 @@
         <material>Gazebo/Blue</material>
     </gazebo>
+    <!-- Gazebo Interface -->
+    <gazebo reference="base_link">
+        <material>Gazebo/Blue</material>
+    </gazebo>
     <!-- Ackerman Steering Macro -->
     <xacro:macro name="ackerman_steering" params="prefix reflect">

Commit message: Updates to mass

File: urdf/basic_pig.urdf.xacro (robot description, xacro)
@@ -32,7 +32,9 @@
     <xacro:property name="front_wheel_width" value=".254" />
     <xacro:property name="front_wheel_diameter" value="0.605" />
+    <xacro:property name="front_wheel_mass" value="9.0"/>
     <!-- Rear Wheel Properties -->
     <xacro:property name="rear_wheel_width" value="0.2794" />
     <xacro:property name="rear_wheel_diameter" value="0.635" />
+    <xacro:property name="rear_wheel_mass" value="9.8"/>
     <!-- Main Body of Little Pig -->
     <link name="base_link">
@@ -175,9 +177,5 @@
                 </geometry>
             </collision>
-            <inertial>
-                <origin xyz="0.0 0.0 0.0" rpy="0.0 0.0 0.0"/>
-                <mass value="20.995"/>
-                <inertia ixx="0.996" ixy="0.0" ixz="0.0" iyy="0.612" iyz="0.0" izz="0.612"/>
-            </inertial>
+            <xacro:default_inertial mass="${rear_wheel_mass}" />
         </link>
         <!-- The Joint -->
@@ -187,16 +185,17 @@
             <child link="rear_${suffix}_wheel"/>
             <origin xyz="-${body_length / 2.5} ${(body_width /2) * reflect} -${(body_height / 5) + (rear_wheel_diameter / 2)}" rpy="0.0 0.0 0.0"/>
+            <limit effort="${axle_eff_limit}" velocity="${axle_vel_limit}"/>
         </joint>
         <!-- Gazebo Interface -->
         <gazebo reference="rear_${suffix}_wheel">
-            <!-- <mu1 value="1.0"/>
+            <mu1 value="1.0"/>
             <mu2 value="1.0"/>
             <kp value="10000000.0" />
             <kd value="1.0" />
-            <fdir1 value="1 0 0"/> -->
+            <fdir1 value="1 0 0"/>
             <material>Gazebo/Black</material>
         </gazebo>
         <!-- The Transmission -->
-        <!-- <transmission name="base_to_rear_${suffix}_wheel_trans">
+        <transmission name="base_to_rear_${suffix}_wheel_trans">
             <type>transmission_interface/SimpleTransmission</type>
             <joint name="base_to_rear_${suffix}_wheel">
@@ -207,5 +206,5 @@
                 <mechanicalReduction>1</mechanicalReduction>
             </actuator>
-        </transmission> -->
+        </transmission>
     </xacro:macro>
     <!-- Call the ackermans in for left/right -->

Commit message: update urdf

File: urdf/basic_pig.urdf.xacro (robot description, xacro)
@@ -25,5 +25,5 @@
     <xacro:property name="body_width" value="0.680618" />
     <xacro:property name="body_height" value="1.065022" />
-    <xacro:property name="body_mass" value="40"/>
+    <xacro:property name="body_mass" value="80"/>
     <!-- The Ackerman Steering Hub -->
     <xacro:property name="ackerman_joint_diameter" value="0.09" />
@@ -32,9 +32,9 @@
     <xacro:property name="front_wheel_width" value=".254" />
     <xacro:property name="front_wheel_diameter" value="0.605" />
-    <xacro:property name="front_wheel_mass" value="9.0"/>
+    <xacro:property name="front_wheel_mass" value="20"/>
     <!-- Rear Wheel Properties -->
     <xacro:property name="rear_wheel_width" value="0.2794" />
     <xacro:property name="rear_wheel_diameter" value="0.635" />
-    <xacro:property name="rear_wheel_mass" value="9.8"/>
+    <xacro:property name="rear_wheel_mass" value="20"/>
     <!-- Main Body of Little Pig -->
     <link name="base_link">
@@ -152,8 +152,8 @@
             <type>transmission_interface/SimpleTransmission</type>
             <joint name="${prefix}_ackerman_link_front_${suffix}_wheel">
-                <hardwareInterface>hardware_interface/VelocityJointInterface</hardwareInterface>
+                <hardwareInterface>hardware_interface/EffortJointInterface</hardwareInterface>
             </joint>
             <actuator name="${prefix}_ackerman_link_front_${suffix}_wheel_motor">
-                <hardwareInterface>hardware_interface/VelocityJointInterface</hardwareInterface>
+                <hardwareInterface>hardware_interface/EffortJointInterface</hardwareInterface>
                 <mechanicalReduction>1</mechanicalReduction>
             </actuator>
@@ -200,8 +200,8 @@
             <type>transmission_interface/SimpleTransmission</type>
             <joint name="base_to_rear_${suffix}_wheel">
-                <hardwareInterface>hardware_interface/VelocityJointInterface</hardwareInterface>
+                <hardwareInterface>hardware_interface/EffortJointInterface</hardwareInterface>
             </joint>
             <actuator name="base_to_rear_${suffix}_wheel_motor">
-                <hardwareInterface>hardware_interface/VelocityJointInterface</hardwareInterface>
+                <hardwareInterface>hardware_interface/EffortJointInterface</hardwareInterface>
                 <mechanicalReduction>1</mechanicalReduction>
             </actuator>
