Commit message: Had to edit some links, joints,properties

File: urdf/basic_pig.urdf.xacro (robot description, xacro)
@@ -1,7 +1,4 @@
 <?xml version="1.0"?>
-<robot name="basic_pig"
-    xmlns:xacro="http://www.ros.org/wiki/xacro">
-    <!-- Standard Params -->
-    <xacro:property name="pi" value="3.1415" />
+<robot xmlns:xacro="http://www.ros.org/wiki/xacro" name="basic_pig">
     <!-- Degree-to-radian conversions -->
     <xacro:property name="degrees_45" value="0.785398163"/>
@@ -15,10 +12,4 @@
         </inertial>
     </xacro:macro>
-    <xacro:property name="axle_eff_limit" value="100"/>
-    <xacro:property name="axle_vel_limit" value="39.02"/>
-    <!-- Servo_stall_torque of the direction axis in Nm. servo_no_load_speed is
-       measured in rad/s. -->
-    <xacro:property name="servo_stall_torque" value="100"/>
-    <xacro:property name="servo_no_load_speed" value="100"/>
     <!-- Basic Geometry of Body -->
     <xacro:property name="body_length" value="1.91" />
@@ -26,16 +17,17 @@
     <xacro:property name="body_height" value="1.065022" />
     <xacro:property name="body_mass" value="80"/>
-    <!-- The Ackerman Steering Hub -->
-    <xacro:property name="ackerman_joint_diameter" value="0.09" />
-    <xacro:property name="ackerman_joint_width" value="0.09" />
     <!-- Front Wheel Properties -->
     <xacro:property name="front_wheel_width" value=".254" />
     <xacro:property name="front_wheel_diameter" value="0.605" />
     <xacro:property name="front_wheel_mass" value="20"/>
+    <!-- Steering Link Properties -->
+    <xacro:property name="steering_width" value="${front_wheel_width/4}" />
+    <xacro:property name="steering_diameter" value="${front_wheel_diameter/5}" />
+    <xacro:property name="steering_mass" value="2"/>
     <!-- Rear Wheel Properties -->
-    <xacro:property name="rear_wheel_width" value="0.2794" />
+    <xacro:property name="rear_wheel_width" value="${front_wheel_width+steering_width}" />
     <xacro:property name="rear_wheel_diameter" value="0.635" />
-    <xacro:property name="rear_wheel_mass" value="20"/>
-    <!-- Main Body of Little Pig -->
+    <xacro:property name="rear_wheel_mass" value="22.8"/>
+    <!-- Base Link -->
     <link name="base_link">
         <visual>
@@ -50,57 +42,37 @@
             </geometry>
         </collision>
-        <xacro:default_inertial mass="${body_mass}" />
+        <xacro:default_inertial mass="${body_mass}"/>
     </link>
-    <!-- Gazebo Interface -->
-    <gazebo reference="base_link">
-        <material>Gazebo/Blue</material>
-    </gazebo>
-    <!-- Gazebo Interface -->
-    <gazebo reference="base_link">
-        <material>Gazebo/Blue</material>
-    </gazebo>
-    <!-- Ackerman Steering Macro -->
-    <xacro:macro name="ackerman_steering" params="prefix reflect">
-        <!-- The Link -->
-        <link name="${prefix}_ackerman_link">
+    <!-- Steering Macro -->
+    <xacro:macro name="steering_link" params="prefix reflect">
+        <link name="${prefix}_steering_link">
             <visual>
-                <origin xyz="0.0 0.0 0.0" rpy="${pi/2} 0.0 0.0"/>
+                <origin xyz="0.0 0.0 0.0" rpy="${degrees_90} 0.0 0.0"/>
                 <geometry>
-                    <cylinder radius="${ackerman_joint_diameter/2}" length="${ackerman_joint_width}"/>
+                    <cylinder radius="${steering_diameter}" length="${steering_width}"/>
                 </geometry>
-                <material name="black" />
             </visual>
             <collision>
-                <origin xyz="0.0 0.0 0.0" rpy="${pi/2} 0.0 0.0"/>
+                <origin xyz="0.0 0.0 0.0" rpy="${degrees_90} 0.0 0.0"/>
                 <geometry>
-                    <cylinder radius="${ackerman_joint_diameter/2}" length="${ackerman_joint_width}"/>
+                    <cylinder radius="${steering_diameter}" length="${steering_width}"/>
                 </geometry>
             </collision>
-            <xacro:default_inertial mass="2"/>
+            <xacro:default_inertial mass="${steering_mass}"/>
         </link>
-        <!-- The Joint -->
-        <joint name="base_link_${prefix}_ackerman_link" type="revolute">
-            <axis xyz="0.0 0.0 1.0" rpy="0.0 0.0 0.0"/>
+        <joint name="${prefix}_steering_joint" type="revolute">
             <parent link="base_link"/>
-            <child link="${prefix}_ackerman_link"/>
-            <origin xyz="${body_length / 2.5} ${((ackerman_joint_width/2) + (body_width/2)) * reflect} -${(body_height / 2.25) + (ackerman_joint_diameter / 2)}" rpy="0.0 0.0 0.0"/>
-            <limit lower="${-degrees_45}" upper="${degrees_45}" effort="${servo_stall_torque}" velocity="${servo_no_load_speed}"/>
+            <child link="${prefix}_steering_link"/>
+            <axis xyz="0.0 0.0 0.1"/>
+            <origin xyz="${(body_length / 2)- 0.1} ${(body_width / 2 + steering_width / 2) * reflect} ${-(body_height/2) + 0.1}" rpy="0.0 0.0 0.0"/>
+            <limit lower="-0.22" upper="0.22" effort="0.0" velocity="0.0"/>
         </joint>
-        <!-- Gazebo Interface -->
-        <gazebo reference="${prefix}_ackerman_link">
-            <mu1 value="1.0"/>
-            <mu2 value="1.0"/>
-            <kp value="10000000.0" />
-            <kd value="1.0" />
-            <fdir1 value="1 0 0"/>
-            <material>Gazebo/Black</material>
-        </gazebo>
         <!-- The Transmission -->
-        <transmission name="base_link_${prefix}_ackerman_link_trans">
+        <transmission name="${prefix}_steering_link_trans">
             <type>transmission_interface/SimpleTransmission</type>
-            <joint name="base_link_${prefix}_ackerman_link">
+            <joint name="${prefix}_steering_joint">
                 <hardwareInterface>hardware_interface/EffortJointInterface</hardwareInterface>
             </joint>
-            <actuator name="base_link_${prefix}_ackerman_link_motor">
+            <actuator name="${prefix}_steering_link_motor">
                 <hardwareInterface>hardware_interface/EffortJointInterface</hardwareInterface>
                 <mechanicalReduction>1</mechanicalReduction>
@@ -109,50 +81,33 @@
     </xacro:macro>
     <!-- Front Wheel Macro -->
-    <xacro:macro name="front_wheel" params="prefix suffix reflect">
-        <!-- The Link -->
-        <link name="front_${suffix}_wheel">
+    <xacro:macro name="front_wheel_link" params="prefix reflect">
+        <link name="${prefix}_front_wheel">
             <visual>
-                <origin xyz="0.0 ${(front_wheel_width/2) * reflect} 0.0" rpy="${pi/2} 0.0 0.0"/>
+                <origin xyz="0.0 0.0 0.0" rpy="${degrees_90} 0.0 0.0"/>
                 <geometry>
                     <cylinder radius="${front_wheel_diameter/2}" length="${front_wheel_width}"/>
                 </geometry>
-                <material name="black" />
             </visual>
             <collision>
-                <origin xyz="0.0 0.0 0.0" rpy="${pi/2} 0.0 0.0"/>
+                <origin xyz="0.0 0.0 0.0" rpy="${degrees_90} 0.0 0.0"/>
                 <geometry>
                     <cylinder radius="${front_wheel_diameter/2}" length="${front_wheel_width}"/>
                 </geometry>
             </collision>
-            <inertial>
-                <origin xyz="0.0 0.0 0.0" rpy="0.0 0.0 0.0"/>
-                <mass value="20.995"/>
-                <inertia ixx="0.996" ixy="0.0" ixz="0.0" iyy="0.612" iyz="0.0" izz="0.612"/>
-            </inertial>
+            <xacro:default_inertial mass="${front_wheel_mass}"/>
         </link>
-        <!-- The Joint -->
-        <joint name="${prefix}_ackerman_link_front_${suffix}_wheel" type="continuous">
-            <axis xyz="0.0 1.0 0.0"/>
-            <parent link="${prefix}_ackerman_link"/>
-            <child link="front_${suffix}_wheel"/>
-            <origin xyz="0.0 0.0 0.0" rpy="0.0 0.0 0.0"/>
-            <limit effort="${axle_eff_limit}" velocity="${axle_vel_limit}"/>
+        <joint name="${prefix}_front_axle" type="continuous">
+            <parent link="${prefix}_steering_link"/>
+            <child link="${prefix}_front_wheel"/>
+            <axis xyz="0.0 0.1 0.0"/>
+            <origin xyz="0 ${(front_wheel_width/2 + steering_width/2) * reflect} 0"/>
         </joint>
-        <!-- Gazebo Interface -->
-        <gazebo reference="front_${suffix}_wheel">
-            <mu1 value="1.0"/>
-            <mu2 value="1.0"/>
-            <kp value="10000000.0" />
-            <kd value="1.0" />
-            <fdir1 value="0 0 1"/>
-            <material>Gazebo/Black</material>
-        </gazebo>
         <!-- The Transmission -->
-        <transmission name="${prefix}_ackerman_link_front_${suffix}_wheel_trans">
+        <transmission name="${prefix}_front_wheel_trans">
             <type>transmission_interface/SimpleTransmission</type>
-            <joint name="${prefix}_ackerman_link_front_${suffix}_wheel">
+            <joint name="${prefix}_front_axle">
                 <hardwareInterface>hardware_interface/EffortJointInterface</hardwareInterface>
             </joint>
-            <actuator name="${prefix}_ackerman_link_front_${suffix}_wheel_motor">
+            <actuator name="${prefix}_front_wheel_motor">
                 <hardwareInterface>hardware_interface/EffortJointInterface</hardwareInterface>
                 <mechanicalReduction>1</mechanicalReduction>
@@ -160,47 +115,34 @@
         </transmission>
     </xacro:macro>
-    <!-- Back Wheel Macro -->
-    <xacro:macro name="rear_wheel" params="suffix reflect">
-        <!-- The Link -->
-        <link name="rear_${suffix}_wheel">
+    <!-- Rear Wheel Macro -->
+    <xacro:macro name="rear_wheel_link" params="prefix reflect">
+        <link name="${prefix}_rear_wheel">
             <visual>
-                <origin xyz="0.0 ${(rear_wheel_width / 2) * reflect} 0.0" rpy="${pi/2} 0.0 0.0"/>
+                <origin xyz="0.0 0.0 0.0" rpy="${degrees_90} 0.0 0.0"/>
                 <geometry>
                     <cylinder radius="${rear_wheel_diameter/2}" length="${rear_wheel_width}"/>
                 </geometry>
-                <material name="black" />
             </visual>
             <collision>
-                <origin xyz="0.0 0.0 0.0" rpy="${pi/2} 0.0 0.0"/>
+                <origin xyz="0.0 0.0 0.0" rpy="${degrees_90} 0.0 0.0"/>
                 <geometry>
                     <cylinder radius="${rear_wheel_diameter/2}" length="${rear_wheel_width}"/>
                 </geometry>
             </collision>
-            <xacro:default_inertial mass="${rear_wheel_mass}" />
+            <xacro:default_inertial mass="${rear_wheel_mass}"/>
         </link>
-        <!-- The Joint -->
-        <joint name="base_to_rear_${suffix}_wheel" type="continuous">
-            <axis xyz="0.0 1.0 0.0"/>
+        <joint name="${prefix}_rear_axle" type="continuous">
             <parent link="base_link"/>
-            <child link="rear_${suffix}_wheel"/>
-            <origin xyz="-${body_length / 2.5} ${(body_width /2) * reflect} -${(body_height / 5) + (rear_wheel_diameter / 2)}" rpy="0.0 0.0 0.0"/>
-            <limit effort="${axle_eff_limit}" velocity="${axle_vel_limit}"/>
+            <child link="${prefix}_rear_wheel"/>
+            <axis xyz="0.0 0.1 0.0"/>
+            <origin xyz="${-(body_length/2) + 0.1} ${(rear_wheel_width/2 + body_width/2) * reflect} ${-(body_height/2) + 0.1}"/>
         </joint>
-        <!-- Gazebo Interface -->
-        <gazebo reference="rear_${suffix}_wheel">
-            <mu1 value="1.0"/>
-            <mu2 value="1.0"/>
-            <kp value="10000000.0" />
-            <kd value="1.0" />
-            <fdir1 value="1 0 0"/>
-            <material>Gazebo/Black</material>
-        </gazebo>
         <!-- The Transmission -->
-        <transmission name="base_to_rear_${suffix}_wheel_trans">
+        <transmission name="${prefix}_rear_wheel_trans">
             <type>transmission_interface/SimpleTransmission</type>
-            <joint name="base_to_rear_${suffix}_wheel">
+            <joint name="${prefix}_rear_axle">
                 <hardwareInterface>hardware_interface/EffortJointInterface</hardwareInterface>
             </joint>
-            <actuator name="base_to_rear_${suffix}_wheel_motor">
+            <actuator name="${prefix}_rear_wheel_motor">
                 <hardwareInterface>hardware_interface/EffortJointInterface</hardwareInterface>
                 <mechanicalReduction>1</mechanicalReduction>
@@ -208,17 +150,14 @@
         </transmission>
     </xacro:macro>
-    <!-- Call the ackermans in for left/right -->
-    <xacro:ackerman_steering prefix="left" reflect="1" />
-    <xacro:ackerman_steering prefix="right" reflect="-1" />
-    <!-- Call the front wheels in left/right -->
-    <xacro:front_wheel prefix="left" suffix="left" reflect="1" />
-    <xacro:front_wheel prefix="right" suffix="right" reflect="-1" />
-    <!-- Call the rear wheels in left/right-->
-    <xacro:rear_wheel suffix="left" reflect="1" />
-    <xacro:rear_wheel suffix="right" reflect="-1" />
+    <xacro:steering_link prefix="left" reflect="1" />
+    <xacro:steering_link prefix="right" reflect="-1" />
+    <xacro:front_wheel_link prefix="left" reflect="1" />
+    <xacro:front_wheel_link prefix="right" reflect="-1" />
+    <xacro:rear_wheel_link prefix="left" reflect="1" />
+    <xacro:rear_wheel_link prefix="right" reflect="-1" />
     <!-- Gazebo plugin for ROS Control -->
     <gazebo>
         <plugin name="gazebo_ros_control" filename="libgazebo_ros_control.so">
-            <robotNamespace>/basic_geometry_pig</robotNamespace>
+            <robotNamespace>/basic_pig</robotNamespace>
         </plugin>
     </gazebo>

Commit message: Had to edit some params

File: urdf/basic_pig.urdf.xacro (robot description, xacro)
@@ -16,5 +16,5 @@
     <xacro:property name="body_width" value="0.680618" />
     <xacro:property name="body_height" value="1.065022" />
-    <xacro:property name="body_mass" value="80"/>
+    <xacro:property name="body_mass" value="20.3"/>
     <!-- Front Wheel Properties -->
     <xacro:property name="front_wheel_width" value=".254" />
@@ -66,5 +66,5 @@
             <axis xyz="0.0 0.0 0.1"/>
             <origin xyz="${(body_length / 2)- 0.1} ${(body_width / 2 + steering_width / 2) * reflect} ${-(body_height/2) + 0.1}" rpy="0.0 0.0 0.0"/>
-            <limit lower="-0.22" upper="0.22" effort="0.0" velocity="0.0"/>
+            <limit lower="-0.30" upper="0.30" effort="100.00" velocity="100.00"/>
         </joint>
         <!-- The Transmission -->

Commit message: XACRO changed for correct controller and new plugin

File: urdf/basic_pig.urdf.xacro (robot description, xacro)
@@ -5,4 +5,9 @@
     <xacro:property name="degrees_90" value="1.57079633"/>
     <xacro:property name="degrees_180" value="3.14159265"/>
+    <!-- vehiclur velocity properties -->
+    <xacro:property name="steering_speed" value="1.0472"/> <!-- units of rad/s -->
+    <xacro:property name="steering_max_angle" value="0.3"/> <!-- units of rad -->
+    <xacro:property name="steering_min_angle" value="-0.3"/> <!-- units of rad -->
+    <xacro:property name="traverse_max_speed" value="4.785"/> <!-- units of m/s -->
     <!-- Inertia Generator -->
     <xacro:macro name="default_inertial" params="mass">
@@ -20,16 +25,19 @@
     <xacro:property name="front_wheel_width" value=".254" />
     <xacro:property name="front_wheel_diameter" value="0.605" />
-    <xacro:property name="front_wheel_mass" value="20"/>
+    <xacro:property name="front_wheel_mass" value="20.0"/>
     <!-- Steering Link Properties -->
     <xacro:property name="steering_width" value="${front_wheel_width/4}" />
     <xacro:property name="steering_diameter" value="${front_wheel_diameter/5}" />
-    <xacro:property name="steering_mass" value="2"/>
+    <xacro:property name="steering_mass" value="2.0"/>
     <!-- Rear Wheel Properties -->
     <xacro:property name="rear_wheel_width" value="${front_wheel_width+steering_width}" />
     <xacro:property name="rear_wheel_diameter" value="0.635" />
     <xacro:property name="rear_wheel_mass" value="22.8"/>
-    <!-- Base Link -->
-    <link name="base_link">
+    <!-- Dummy Base Link -->
+    <link name="base_link" />
+    <!-- Actual Base Link -->
+    <link name="chassis">
         <visual>
+            <origin xyz="0.0 0.0 0.0" rpy="0.0 0.0 0.0"/>
             <geometry>
                 <box size="${body_length} ${body_width} ${body_height}"/>
@@ -38,4 +46,5 @@
         </visual>
         <collision>
+            <origin xyz="0.0 0.0 0.0" rpy="0.0 0.0 0.0"/>
             <geometry>
                 <box size="${body_length} ${body_width} ${body_height}"/>
@@ -44,4 +53,9 @@
         <xacro:default_inertial mass="${body_mass}"/>
     </link>
+    <joint name="base_link_joint" type="fixed">
+        <origin xyz="0 0 0.05" rpy="0 0 0" />
+        <parent link="base_link" />
+        <child link="chassis" />
+    </joint>
     <!-- Steering Macro -->
     <xacro:macro name="steering_link" params="prefix reflect">
@@ -62,9 +76,10 @@
         </link>
         <joint name="${prefix}_steering_joint" type="revolute">
-            <parent link="base_link"/>
+            <parent link="chassis"/>
             <child link="${prefix}_steering_link"/>
             <axis xyz="0.0 0.0 0.1"/>
             <origin xyz="${(body_length / 2)- 0.1} ${(body_width / 2 + steering_width / 2) * reflect} ${-(body_height/2) + 0.1}" rpy="0.0 0.0 0.0"/>
-            <limit lower="-0.30" upper="0.30" effort="100.00" velocity="100.00"/>
+            <limit lower="${steering_min_angle}" upper="${steering_max_angle}" effort="100000.00" velocity="${steering_speed}"/>
+            <!-- effort needs to be very high so we are not constrained by the environment-->
         </joint>
         <!-- The Transmission -->
@@ -72,8 +87,8 @@
             <type>transmission_interface/SimpleTransmission</type>
             <joint name="${prefix}_steering_joint">
-                <hardwareInterface>hardware_interface/EffortJointInterface</hardwareInterface>
+                <hardwareInterface>hardware_interface/PositionJointInterface</hardwareInterface>
             </joint>
             <actuator name="${prefix}_steering_link_motor">
-                <hardwareInterface>hardware_interface/EffortJointInterface</hardwareInterface>
+                <hardwareInterface>hardware_interface/PositionJointInterface</hardwareInterface>
                 <mechanicalReduction>1</mechanicalReduction>
             </actuator>
@@ -102,4 +117,6 @@
             <axis xyz="0.0 0.1 0.0"/>
             <origin xyz="0 ${(front_wheel_width/2 + steering_width/2) * reflect} 0"/>
+            <limit effort="100000.00" velocity="${traverse_max_speed * 2 / front_wheel_diameter}"/> <!-- units of rad/s -->
+            <!-- effort needs to be very high so we are not constrained by the environment-->
         </joint>
         <!-- The Transmission -->
@@ -107,8 +124,8 @@
             <type>transmission_interface/SimpleTransmission</type>
             <joint name="${prefix}_front_axle">
-                <hardwareInterface>hardware_interface/EffortJointInterface</hardwareInterface>
+                <hardwareInterface>hardware_interface/VelocityJointInterface</hardwareInterface>
             </joint>
             <actuator name="${prefix}_front_wheel_motor">
-                <hardwareInterface>hardware_interface/EffortJointInterface</hardwareInterface>
+                <hardwareInterface>hardware_interface/VelocityJointInterface</hardwareInterface>
                 <mechanicalReduction>1</mechanicalReduction>
             </actuator>
@@ -133,8 +150,10 @@
         </link>
         <joint name="${prefix}_rear_axle" type="continuous">
-            <parent link="base_link"/>
+            <parent link="chassis"/>
             <child link="${prefix}_rear_wheel"/>
             <axis xyz="0.0 0.1 0.0"/>
             <origin xyz="${-(body_length/2) + 0.1} ${(rear_wheel_width/2 + body_width/2) * reflect} ${-(body_height/2) + 0.1}"/>
+            <limit effort="0.0" velocity="${traverse_max_speed / rear_wheel_diameter}"/> <!-- rolling axle -->
+            <!-- <limit effort="100000.00" velocity="${traverse_max_speed / rear_wheel_diameter}"/> -->
         </joint>
         <!-- The Transmission -->
@@ -142,7 +161,9 @@
             <type>transmission_interface/SimpleTransmission</type>
             <joint name="${prefix}_rear_axle">
+                <!-- <hardwareInterface>hardware_interface/VelocityJointInterface</hardwareInterface> --> <!-- rolling axle -->
                 <hardwareInterface>hardware_interface/EffortJointInterface</hardwareInterface>
             </joint>
             <actuator name="${prefix}_rear_wheel_motor">
+                <!-- <hardwareInterface>hardware_interface/VelocityJointInterface</hardwareInterface> --> <!-- rolling axle -->
                 <hardwareInterface>hardware_interface/EffortJointInterface</hardwareInterface>
                 <mechanicalReduction>1</mechanicalReduction>
@@ -160,4 +181,5 @@
         <plugin name="gazebo_ros_control" filename="libgazebo_ros_control.so">
             <robotNamespace>/basic_pig</robotNamespace>
+            <robotSimType>gazebo_ros_control/AckermannRobotHWSim</robotSimType> <!-- THIS IS NEW -->
         </plugin>
     </gazebo>

Commit message: Description CHanges

File: urdf/basic_pig.urdf.xacro (robot description, xacro)
@@ -2,4 +2,5 @@
 <robot xmlns:xacro="http://www.ros.org/wiki/xacro" name="basic_pig">
     <!-- Degree-to-radian conversions -->
+    <xacro:property name="degrees_30" value="0.523598776"/>
     <xacro:property name="degrees_45" value="0.785398163"/>
     <xacro:property name="degrees_90" value="1.57079633"/>
@@ -7,6 +8,6 @@
     <!-- vehicular velocity properties -->
     <xacro:property name="steering_speed" value="1.0472"/> <!-- units of rad/s -->
-    <xacro:property name="steering_max_angle" value="0.3"/> <!-- units of rad -->
-    <xacro:property name="steering_min_angle" value="-0.3"/> <!-- units of rad -->
+    <xacro:property name="steering_max_angle" value="${degrees_30}"/> <!-- units of rad -->
+    <xacro:property name="steering_min_angle" value="- ${degrees_30}"/> <!-- units of rad -->
     <xacro:property name="traverse_max_speed" value="4.785"/> <!-- units of m/s -->
     <!-- Inertia Generator -->
