Commit message: Major URDF update including shocks for rear

File: urdf/basic_laser_pig_old.urdf.xacro (robot description, xacro)
@@ -2,5 +2,4 @@
 <robot xmlns:xacro="http://www.ros.org/wiki/xacro" name="basic_laser_pig">
     <!-- Degree-to-radian conversions -->
-    <xacro:property name="degrees_30" value="0.523598776"/>
     <xacro:property name="degrees_45" value="0.785398163"/>
     <xacro:property name="degrees_90" value="1.57079633"/>
@@ -8,7 +7,7 @@
     <!-- vehiclur velocity properties -->
     <xacro:property name="steering_speed" value="1.0472"/> <!-- units of rad/s -->
-    <xacro:property name="steering_max_angle" value="${degrees_30}"/> <!-- units of rad -->
-    <xacro:property name="steering_min_angle" value="-${degrees_30}"/> <!-- units of rad -->
-    <xacro:property name="traverse_max_speed" value="4.785"/> <!-- units of m/s 4.785-->
+    <xacro:property name="steering_max_angle" value="0.3"/> <!-- units of rad -->
+    <xacro:property name="steering_min_angle" value="-0.3"/> <!-- units of rad -->
+    <xacro:property name="traverse_max_speed" value="4.785"/> <!-- units of m/s -->
     <!-- Inertia Generator -->
     <xacro:macro name="default_inertial" params="mass">
@@ -22,9 +21,9 @@
     <xacro:property name="body_width" value="0.680618" />
     <xacro:property name="body_height" value="1.065022" />
-    <xacro:property name="body_mass" value="200.0"/>
+    <xacro:property name="body_mass" value="20.3"/>
     <!-- Front Wheel Properties -->
     <xacro:property name="front_wheel_width" value=".254" />
     <xacro:property name="front_wheel_diameter" value="0.605" />
-    <xacro:property name="front_wheel_mass" value="10"/>
+    <xacro:property name="front_wheel_mass" value="20"/>
     <!-- Steering Link Properties -->
     <xacro:property name="steering_width" value="${front_wheel_width/4}" />
@@ -34,5 +33,5 @@
     <xacro:property name="rear_wheel_width" value="${front_wheel_width+steering_width}" />
     <xacro:property name="rear_wheel_diameter" value="0.635" />
-    <xacro:property name="rear_wheel_mass" value="12"/>
+    <xacro:property name="rear_wheel_mass" value="22.8"/>
     <!-- Camera Properties -->
     <xacro:property name="camera_link" value="0.04"/>
@@ -44,5 +43,5 @@
     <link name="chassis">
         <visual>
-            <origin xyz="${(body_length/2) - 0.1} 0.0 0.0" rpy="0.0 0.0 0.0"/>
+            <origin xyz="0.0 0.0 0.0" rpy="0.0 0.0 0.0"/>
             <geometry>
                 <box size="${body_length} ${body_width} ${body_height}"/>
@@ -51,5 +50,5 @@
         </visual>
         <collision>
-            <origin xyz="${(body_length/2) - 0.1} 0.0 0.0" rpy="0.0 0.0 0.0"/>
+            <origin xyz="0.0 0.0 0.0" rpy="0.0 0.0 0.0"/>
             <geometry>
                 <box size="${body_length} ${body_width} ${body_height}"/>
@@ -66,5 +65,5 @@
     <joint name="laser_link_joint" type="fixed">
       <axis xyz="0 0 0" />
-      <origin xyz="${(body_length) + 0.1} 0.0 0.0" rpy="0 0 0"/>
+      <origin xyz="${(body_length/2) - 0.1} 0.0 ${(body_height/2 + 0.1)}" rpy="0 0 0"/>
       <parent link="chassis"/>
       <child link="laser_link"/>
@@ -93,5 +92,5 @@
     <joint name="camera_link_joint" type="fixed">
       <axis xyz="0 1 0" />
-      <origin xyz="${(body_length) - 0.1} 0.0 ${(body_height/2 + 0.2)}" rpy="0 0 0"/>
+      <origin xyz="${(body_length/2) - 0.1} 0.0 ${(body_height/2 + 0.2)}" rpy="0 0 0"/>
       <parent link="chassis"/>
       <child link="camera_link"/>
@@ -101,5 +100,5 @@
         <origin xyz="0 0 0" rpy="0 0 0"/>
         <geometry>
-        <box size="${camera_link} ${camera_link} ${camera_link}"/>
+      <box size="${camera_link} ${camera_link} ${camera_link}"/>
         </geometry>
       </collision>
@@ -107,5 +106,5 @@
         <origin xyz="0 0 0" rpy="0 0 0"/>
         <geometry>
-        <box size="${camera_link} ${camera_link} ${camera_link}"/>
+      <box size="${camera_link} ${camera_link} ${camera_link}"/>
         </geometry>
         <material name="red"/>
@@ -119,29 +118,29 @@
     <!-- IMU -->
     <joint name="imu_joint" type="fixed">
-        <axis xyz="1 0 0 "/> <!-- 0 1 0 -->
-        <origin xyz="0 0 0.19"/>
-        <parent link ="chassis"/>
-        <child link ="imu_link"/>
+      <axis xyz="1 0 0 "/> <!-- 0 1 0 -->
+      <origin xyz="0 0 0.19"/>
+      <parent link ="chassis"/>
+      <child link ="imu_link"/>
     </joint>
     <link name="imu_link">
-        <inertial>
-            <mass value="0.001"/>
-            <origin rpy="0 0 0" xyz="0 0 0"/>
-            <inertia ixx="0.0001" ixy="0" ixz="0" iyy="0.000001" iyz="0" izz="0.0001"/>
-        </inertial>
-        <visual>
-            <origin rpy="0 0 0" xyz="0 0 0"/>
-            <geometry>
-            <box size="0.001 0.001 0.001"/>
-            </geometry>
-        </visual>
-        <collision>
-            <origin rpy="0 0 0" xyz="0 0 0"/>
-            <geometry>
-            <box size=".001 .001 .001"/>
-            </geometry>
-        </collision>
+	<inertial>
+	    <mass value="0.001"/>
+	    <origin rpy="0 0 0" xyz="0 0 0"/>
+	    <inertia ixx="0.0001" ixy="0" ixz="0" iyy="0.000001" iyz="0" izz="0.0001"/>
+	</inertial>
+	<visual>
+	    <origin rpy="0 0 0" xyz="0 0 0"/>
+	    <geometry>
+	      <box size="0.001 0.001 0.001"/>
+	    </geometry>
+	</visual>
+	  <collision>
+	    <origin rpy="0 0 0" xyz="0 0 0"/>
+	    <geometry>
+	      <box size=".001 .001 .001"/>
+	    </geometry>
+	  </collision>
 	</link>
-    <!-- GPS (THIS JOINT IS UNNECESSARY)
+    <!-- GPS -->
     <joint name="gps_joint" type="fixed">
       <axis xyz="0 0 0 "/>
@@ -151,23 +150,22 @@
     </joint>
     <link name="gps_link">
-        <inertial>
-            <mass value="0.001"/>
-            <origin rpy="0 0 0" xyz="0 0 0"/>
-            <inertia ixx="0.0001" ixy="0" ixz="0" iyy="0.000001" iyz="0" izz="0.0001"/>
-        </inertial>
-        <visual>
-            <origin rpy="0 0 0" xyz="0 0 0"/>
-            <geometry>
-            <box size="0.001 0.001 0.001"/>
-            </geometry>
-        </visual>
-        <collision>
-            <origin rpy="0 0 0" xyz="0 0 0"/>
-            <geometry>
-            <box size=".001 .001 .001"/>
-            </geometry>
-        </collision>
+	<inertial>
+	    <mass value="0.001"/>
+	    <origin rpy="0 0 0" xyz="0 0 0"/>
+	    <inertia ixx="0.0001" ixy="0" ixz="0" iyy="0.000001" iyz="0" izz="0.0001"/>
+	</inertial>
+	<visual>
+	    <origin rpy="0 0 0" xyz="0 0 0"/>
+	    <geometry>
+	      <box size="0.001 0.001 0.001"/>
+	    </geometry>
+	</visual>
+	  <collision>
+	    <origin rpy="0 0 0" xyz="0 0 0"/>
+	    <geometry>
+	      <box size=".001 .001 .001"/>
+	    </geometry>
+	  </collision>
 	</link>
-    -->
     <!-- Steering Macro -->
     <xacro:macro name="steering_link" params="prefix reflect">
@@ -191,5 +189,5 @@
             <child link="${prefix}_steering_link"/>
             <axis xyz="0.0 0.0 0.1"/>
-            <origin xyz="${(body_length)- 0.2} ${(body_width / 2 + steering_width / 2 + 0.1) * reflect} ${-(body_height/2) + 0.1}" rpy="0.0 0.0 0.0"/>
+            <origin xyz="${(body_length / 2)- 0.1} ${(body_width / 2 + steering_width / 2 + 0.1) * reflect} ${-(body_height/2) + 0.1}" rpy="0.0 0.0 0.0"/>
             <limit lower="${steering_min_angle}" upper="${steering_max_angle}" effort="100000.00" velocity="${steering_speed}"/>
             <!-- effort needs to be very high so we are not constrained by the environment-->
@@ -219,30 +217,30 @@
                 <origin xyz="0.0 0.0 0.0" rpy="${degrees_90} 0.0 0.0"/>
                 <geometry>
-                    <cylinder radius="${front_wheel_diameter/2}" length="0.02"/>
-                </geometry>
-                    <surface>
-                        <friction>
-                            <torsional>
-                                <coefficient>2.0</coefficient>
-                                <surface_radius>.3025</surface_radius>
-                                <use_patch_radius>false</use_patch_radius>
-                                <ode>
-                                    <slip>0.5</slip>
-                                </ode>
-                            </torsional>
-                            <ode>
-                                <mu>50000.00</mu>
-                                <mu2>50000.00</mu2>
-                                <fdir1>1.00000 0.00000 0.00000</fdir1>
-                                <slip1>0.00000</slip1>
-                                <slip2>0.00000</slip2>
-                            </ode>
-                        </friction>
-                        <contact>
-                            <ode>
-                                <min_depth>0.03</min_depth>
-                            </ode>
-                        </contact>
-                    </surface>
+                    <cylinder radius="${front_wheel_diameter/2}" length="${front_wheel_width}"/>
+                </geometry>
+		<surface>
+			<friction>
+				<torsional>
+					<coefficient>2.0</coefficient>
+					<surface_radius>.3025</surface_radius>
+					<use_patch_radius>false</use_patch_radius>
+					<ode>
+						<slip>0.5</slip>
+					</ode>
+				</torsional>
+				<ode>
+					<mu>50000.00</mu>
+					<mu2>50000.00</mu2>
+					<fdir1>1.00000 0.00000 0.00000</fdir1>
+					<slip1>0.00000</slip1>
+					<slip2>0.00000</slip2>
+				</ode>
+			</friction>
+			<contact>
+				<ode>
+					<min_depth>0.03</min_depth>
+				</ode>
+			</contact>
+		</surface>
             </collision>
             <xacro:default_inertial mass="${front_wheel_mass}"/>
@@ -268,33 +266,4 @@
         </transmission>
     </xacro:macro>
-    <!-- Rear Wheel Prismatic Link Macro -->
-    <xacro:macro name="rear_wheel_strut_link" params="prefix reflect">
-        <link name="${prefix}_rear_wheel_strut">
-            <visual>
-                <origin xyz="0.0 0.0 0.0" rpy="${degrees_90} 0.0 0.0"/>
-                <geometry>
-                    <cylinder radius="0.1" length="0.02"/>
-                </geometry>
-            </visual>
-            <collision>
-                <origin xyz="0.0 0.0 0.0" rpy="${degrees_90} 0.0 0.0"/>
-                <geometry>
-                    <cylinder radius="0.1" length="0.02"/>
-                </geometry>
-            </collision>
-            <xacro:default_inertial mass="${rear_wheel_mass}"/>
-        </link>
-        <joint name="${prefix}_rear_strut}" type="prismatic">
-            <parent link="chassis"/>
-            <child link="${prefix}_rear_wheel_strut"/>
-            <axis xyz="0.0 0.0 0.1"/>
-            <origin xyz="0.0 ${(body_width/2 + 0.1) * reflect} ${-(body_height/2) + 0.1}"/>
-            <limit lower="-0.05" upper="0.05" effort="1000.0" velocity="1.0"/>
-            <dynamics damping="2.0" friction="8000.0"/>
-        </joint>
-        <gazebo reference="${prefix}_rear_strut}">
-            <implicitSpringDamper>true</implicitSpringDamper>
-        </gazebo>
-    </xacro:macro>
     <!-- Rear Wheel Macro -->
     <xacro:macro name="rear_wheel_link" params="prefix reflect">
@@ -309,28 +278,46 @@
                 <origin xyz="0.0 0.0 0.0" rpy="${degrees_90} 0.0 0.0"/>
                 <geometry>
-                    <cylinder radius="${rear_wheel_diameter/2}" length="0.02"/>
-                </geometry>
+                    <!-- <cylinder radius="${rear_wheel_diameter/2}" length="${rear_wheel_width}"/> -->
+                    <cylinder radius="${rear_wheel_diameter/2}" length="0.04"/>
+                </geometry>
+		<!-- <surface>
+			<friction>
+				<torsional>
+					<coefficient>2.0</coefficient>
+					<surface_radius>.3175</surface_radius>
+					<use_patch_radius>false</use_patch_radius>
+					<ode>
+						<slip>0.5</slip>
+					</ode>
+				</torsional>
+				<ode>
+					<mu>50000.00</mu>
+					<mu2>50000.00</mu2>
+					<fdir1>1.00000 0.00000 0.00000</fdir1>
+					<slip1>0.00000</slip1>
+					<slip2>0.00000</slip2>
+				</ode>
+			</friction>
+			<contact>
+				<ode>
+					<min_depth>0.03</min_depth>
+				</ode>
+			</contact>
+		</surface> -->
             </collision>
-            <surface>
-                <contact>
-                    <ode>
-                        <min_depth>0.01</min_depth>
-                    </ode>
-                </contact>
-                <friction>
-                    <ode>
-                        <mu>1</mu>
-                        <mu2>1</mu2>
-                        <fdir1>1.0 0 0</fdir1>
-                    </ode>
-                </friction>
-            </surface>
             <xacro:default_inertial mass="${rear_wheel_mass}"/>
         </link>
+        <gazebo reference="{prefix}_rear_wheel">
+          <mu1 value="1.0"/>
+          <mu2 value="1.0"/>
+          <kp value="1000000000.0"/>
+          <kd value="1.0"/>
+          <fdir1 value="1 0 0"/>
+        </gazebo>
         <joint name="${prefix}_rear_axle" type="continuous">
-            <parent link="${prefix}_rear_wheel_strut"/>
+            <parent link="chassis"/>
             <child link="${prefix}_rear_wheel"/>
             <axis xyz="0.0 0.1 0.0"/>
-            <origin xyz="0.0 ${(rear_wheel_width/2) * reflect} 0.0"/>
+            <origin xyz="${-(body_length/2) + 0.1} ${(rear_wheel_width/2 + body_width/2 + 0.1) * reflect} ${-(body_height/2) + 0.1}"/>
             <!-- <limit effort="0.0" velocity="${traverse_max_speed / rear_wheel_diameter}"/> --> <!-- rolling axle -->
             <!-- <limit effort="100000.00" velocity="${traverse_max_speed / rear_wheel_diameter}"/> -->
@@ -354,6 +341,4 @@
     <xacro:front_wheel_link prefix="left" reflect="1" />
     <xacro:front_wheel_link prefix="right" reflect="-1" />
-    <xacro:rear_wheel_strut_link prefix="left" reflect="1"/>
-    <xacro:rear_wheel_strut_link prefix="right" reflect="-1"/>
     <xacro:rear_wheel_link prefix="left" reflect="1" />
     <xacro:rear_wheel_link prefix="right" reflect="-1" />
@@ -361,15 +346,14 @@
     <gazebo>
         <plugin name="gazebo_ros_control" filename="libgazebo_ros_control.so">
-            <robotSimType>gazebo_ros_control/AckermannRobotHWSim</robotSimType>
+            <!-- <robotNamespace></robotNamespace> -->
+            <robotSimType>gazebo_ros_control/AckermannRobotHWSim</robotSimType> <!-- THIS IS NEW -->
         </plugin>
         <plugin name="imu_plugin" filename="libhector_gazebo_ros_imu.so">
             <alwaysOn>true</alwaysOn>
             <bodyName>chassis</bodyName>
-            <topicName>imu/data</topicName>
-            <serviceName>imu/is_calibrated</serviceName>
+            <topicName>imu</topicName>
+            <serviceName>imu_service</serviceName>
             <gaussianNoise>0.0</gaussianNoise>
             <updateRate>20.0</updateRate>
-            <xyzOffsets>0 0 0</xyzOffsets>
-            <rpyOffsets>0 0 0</rpyOffsets>
         </plugin>
         <plugin name="gps_plugin" filename="libhector_gazebo_ros_gps.so">
@@ -379,7 +363,8 @@
             <topicname>fix</topicname>
             <velocitytopicname>fix_vel</velocitytopicname>
+            <!-- <drift>5.0 5.0 5.0</drift>
             <gaussiannoise>0.1 0.1 0.1 </gaussiannoise>
             <velocitydrift>0 0 0</velocitydrift>
-            <velocitygaussiannoise>0.1 0.1 0.1</velocitygaussiannoise>
+            <velocitygaussiannoise>0.1 0.1 0.1</velocitygaussiannoise> -->
             <referenceLatitude>37.634047</referenceLatitude>
             <referenceLongitude>-97.269368</referenceLongitude>
