Commit message: added laser sim to little pig

File: urdf/basic_laser_pig.urdf.xacro (robot description, xacro)
@@ -29,4 +29,6 @@
     <xacro:property name="rear_wheel_diameter" value="0.635" />
     <xacro:property name="rear_wheel_mass" value="22.8"/>
+    <!-- Testing Laser link xacro -->
+    <xacro:include filename="$(find little_pig_description)/urdf/basic_laser_pig.gazebo" />
     <!-- Base Link -->
     <link name="base_link">
@@ -44,5 +46,5 @@
         <xacro:default_inertial mass="${body_mass}"/>
     </link>
-    <!-- Laser Link -->
+    <!-- Laser Link
     <link name="laser_link">
       <visual>
@@ -64,40 +66,32 @@
       <axis xyz="0.0 0.0 0.0"/>
       <origin xyz="${(body_length/2) - 0.1} 0.0 ${(body_height/2 + 0.1)}" />
+    </joint> -->
+    <!-- Testing laser link -->
+    <joint name="laser_link_joint" type="fixed">
+      <axis xyz="0 0 0" />
+      <origin xyz="${(body_length/2) - 0.1} 0.0 ${(body_height/2 + 0.1)}" rpy="0 0 0"/>
+      <parent link="base_link"/>
+      <child link="laser_link"/>
     </joint>
-    <gazebo reference="laser_link">
-      <sensor type="gpu_ray" name="head_hokuyo_sensor">
-        <pose>0 0 0 0 0 0</pose>
-        <visualize>true</visualize>
-        <update_rate>40</update_rate>
-        <ray>
-          <scan>
-            <horizontal>
-              <samples>720</samples>
-              <resolution>1</resolution>
-              <min_angle>-1.570796</min_angle>
-              <max_angle>1.570796</max_angle>
-            </horizontal>
-          </scan>
-          <range>
-            <min>0.10</min>
-            <max>30.0</max>
-            <resolution>0.01</resolution>
-          </range>
-          <noise>
-            <type>gaussian</type>
-            <!-- Noise parameters based on published spec for Hokuyo laser
-                 achieving "+-30mm" accuracy at range < 10m.  A mean of 0.0m and
-                 stddev of 0.01m will put 99.7% of samples within 0.03m of the true
-                 reading. -->
-            <mean>0.0</mean>
-            <stddev>0.01</stddev>
-          </noise>
-        </ray>
-        <plugin name="gazebo_ros_head_hokuyo_controller" filename="libgazebo_ros_gpu_laser.so">
-          <topicName>/basic_laser_pig/laser/scan</topicName>
-          <frameName>laser_link</frameName>
-        </plugin>
-      </sensor>
-    </gazebo>
+     <!-- Hokuyo Laser -->
+    <link name="laser_link">
+      <collision>
+        <origin xyz="0 0 0" rpy="0 0 0"/>
+        <geometry>
+          <cylinder radius=".05" length="0.04"/>
+        </geometry>
+      </collision>
+      <visual>
+        <origin xyz="0 0 0" rpy="0 0 0"/>
+        <geometry>
+          <cylinder radius=".05" length="0.04"/>
+        </geometry>
+      </visual>
+      <inertial>
+        <mass value="1e-5" />
+        <origin xyz="0 0 0" rpy="0 0 0"/>
+        <inertia ixx="1e-6" ixy="0" ixz="0" iyy="1e-6" iyz="0" izz="1e-6" />
+      </inertial>
+    </link>
     <!-- Steering Macro -->
     <xacro:macro name="steering_link" params="prefix reflect">

Commit message: added camera NOT POINT CLOUD

File: urdf/basic_laser_pig.urdf.xacro (robot description, xacro)
@@ -29,4 +29,6 @@
     <xacro:property name="rear_wheel_diameter" value="0.635" />
     <xacro:property name="rear_wheel_mass" value="22.8"/>
+    <!-- Camera Properties -->
+    <xacro:property name="camera_link" value="0.04"/>
     <!-- Testing Laser link xacro -->
     <xacro:include filename="$(find little_pig_description)/urdf/basic_laser_pig.gazebo" />
@@ -46,26 +48,5 @@
         <xacro:default_inertial mass="${body_mass}"/>
     </link>
-    <!-- Laser Link
-    <link name="laser_link">
-      <visual>
-        <origin xyz="0.0 0.0 0.0" rpy="0.0 0.0 0.0"/>
-        <geometry>
-          <cylinder radius=".05" length="0.04"/>
-        </geometry>
-      </visual>
-      <collision>
-        <geometry>
-          <cylinder radius=".05" length="0.04"/>
-        </geometry>
-      </collision>
-      <xacro:default_inertial mass="0.01"/>
-    </link>
-    <joint name="base_link_laser_link" type="fixed">
-      <parent link="base_link"/>
-      <child link="laser_link"/>
-      <axis xyz="0.0 0.0 0.0"/>
-      <origin xyz="${(body_length/2) - 0.1} 0.0 ${(body_height/2 + 0.1)}" />
-    </joint> -->
-    <!-- Testing laser link -->
+    <!-- Laser link -->
     <joint name="laser_link_joint" type="fixed">
       <axis xyz="0 0 0" />
@@ -74,5 +55,5 @@
       <child link="laser_link"/>
     </joint>
-     <!-- Hokuyo Laser -->
+     <!-- Laser -->
     <link name="laser_link">
       <collision>
@@ -87,4 +68,31 @@
           <cylinder radius=".05" length="0.04"/>
         </geometry>
+      </visual>
+      <inertial>
+        <mass value="1e-5" />
+        <origin xyz="0 0 0" rpy="0 0 0"/>
+        <inertia ixx="1e-6" ixy="0" ixz="0" iyy="1e-6" iyz="0" izz="1e-6" />
+      </inertial>
+    </link>
+    <!-- Camera -->
+    <joint name="camera_link_joint" type="fixed">
+      <axis xyz="0 1 0" />
+      <origin xyz="${(body_length/2) - 0.1} 0.0 ${(body_height/2 + 0.2)}" rpy="0 0 0"/>
+      <parent link="base_link"/>
+      <child link="camera_link"/>
+    </joint>
+    <link name="camera_link">
+      <collision>
+        <origin xyz="0 0 0" rpy="0 0 0"/>
+        <geometry>
+      <box size="${camera_link} ${camera_link} ${camera_link}"/>
+        </geometry>
+      </collision>
+      <visual>
+        <origin xyz="0 0 0" rpy="0 0 0"/>
+        <geometry>
+      <box size="${camera_link} ${camera_link} ${camera_link}"/>
+        </geometry>
+        <material name="red"/>
       </visual>
       <inertial>

Commit message: Updated Laser Pig

File: urdf/basic_laser_pig.urdf.xacro (robot description, xacro)
@@ -5,4 +5,9 @@
     <xacro:property name="degrees_90" value="1.57079633"/>
     <xacro:property name="degrees_180" value="3.14159265"/>
+    <!-- vehiclur velocity properties -->
+    <xacro:property name="steering_speed" value="1.0472"/> <!-- units of rad/s -->
+    <xacro:property name="steering_max_angle" value="0.3"/> <!-- units of rad -->
+    <xacro:property name="steering_min_angle" value="-0.3"/> <!-- units of rad -->
+    <xacro:property name="traverse_max_speed" value="4.785"/> <!-- units of m/s -->
     <!-- Inertia Generator -->
     <xacro:macro name="default_inertial" params="mass">
@@ -33,7 +38,10 @@
     <!-- Testing Laser link xacro -->
     <xacro:include filename="$(find little_pig_description)/urdf/basic_laser_pig.gazebo" />
-    <!-- Base Link -->
-    <link name="base_link">
+    <!-- Dummy Base Link -->
+    <link name="base_link" />
+    <!-- Actual Base Link -->
+    <link name="chassis">
         <visual>
+            <origin xyz="0.0 0.0 0.0" rpy="0.0 0.0 0.0"/>
             <geometry>
                 <box size="${body_length} ${body_width} ${body_height}"/>
@@ -42,4 +50,5 @@
         </visual>
         <collision>
+            <origin xyz="0.0 0.0 0.0" rpy="0.0 0.0 0.0"/>
             <geometry>
                 <box size="${body_length} ${body_width} ${body_height}"/>
@@ -48,9 +57,14 @@
         <xacro:default_inertial mass="${body_mass}"/>
     </link>
+    <joint name="base_link_joint" type="fixed">
+        <origin xyz="0 0 0.05" rpy="0 0 0" />
+        <parent link="base_link" />
+        <child link="chassis" />
+    </joint>
     <!-- Laser link -->
     <joint name="laser_link_joint" type="fixed">
       <axis xyz="0 0 0" />
       <origin xyz="${(body_length/2) - 0.1} 0.0 ${(body_height/2 + 0.1)}" rpy="0 0 0"/>
-      <parent link="base_link"/>
+      <parent link="chassis"/>
       <child link="laser_link"/>
     </joint>
@@ -79,5 +93,5 @@
       <axis xyz="0 1 0" />
       <origin xyz="${(body_length/2) - 0.1} 0.0 ${(body_height/2 + 0.2)}" rpy="0 0 0"/>
-      <parent link="base_link"/>
+      <parent link="chassis"/>
       <child link="camera_link"/>
     </joint>
@@ -120,9 +134,10 @@
         </link>
         <joint name="${prefix}_steering_joint" type="revolute">
-            <parent link="base_link"/>
+            <parent link="chassis"/>
             <child link="${prefix}_steering_link"/>
             <axis xyz="0.0 0.0 0.1"/>
             <origin xyz="${(body_length / 2)- 0.1} ${(body_width / 2 + steering_width / 2) * reflect} ${-(body_height/2) + 0.1}" rpy="0.0 0.0 0.0"/>
-            <limit lower="-0.30" upper="0.30" effort="100.00" velocity="100.00"/>
+            <limit lower="${steering_min_angle}" upper="${steering_max_angle}" effort="100000.00" velocity="${steering_speed}"/>
+            <!-- effort needs to be very high so we are not constrained by the environment-->
         </joint>
         <!-- The Transmission -->
@@ -130,8 +145,8 @@
             <type>transmission_interface/SimpleTransmission</type>
             <joint name="${prefix}_steering_joint">
-                <hardwareInterface>hardware_interface/EffortJointInterface</hardwareInterface>
+                <hardwareInterface>hardware_interface/PositionJointInterface</hardwareInterface>
             </joint>
             <actuator name="${prefix}_steering_link_motor">
-                <hardwareInterface>hardware_interface/EffortJointInterface</hardwareInterface>
+                <hardwareInterface>hardware_interface/PositionJointInterface</hardwareInterface>
                 <mechanicalReduction>1</mechanicalReduction>
             </actuator>
@@ -160,4 +175,6 @@
             <axis xyz="0.0 0.1 0.0"/>
             <origin xyz="0 ${(front_wheel_width/2 + steering_width/2) * reflect} 0"/>
+            <limit effort="100000.00" velocity="${traverse_max_speed * 2 / front_wheel_diameter}"/> <!-- units of rad/s -->
+            <!-- effort needs to be very high so we are not constrained by the environment-->
         </joint>
         <!-- The Transmission -->
@@ -165,8 +182,8 @@
             <type>transmission_interface/SimpleTransmission</type>
             <joint name="${prefix}_front_axle">
-                <hardwareInterface>hardware_interface/EffortJointInterface</hardwareInterface>
+                <hardwareInterface>hardware_interface/VelocityJointInterface</hardwareInterface>
             </joint>
             <actuator name="${prefix}_front_wheel_motor">
-                <hardwareInterface>hardware_interface/EffortJointInterface</hardwareInterface>
+                <hardwareInterface>hardware_interface/VelocityJointInterface</hardwareInterface>
                 <mechanicalReduction>1</mechanicalReduction>
             </actuator>
@@ -191,8 +208,10 @@
         </link>
         <joint name="${prefix}_rear_axle" type="continuous">
-            <parent link="base_link"/>
+            <parent link="chassis"/>
             <child link="${prefix}_rear_wheel"/>
             <axis xyz="0.0 0.1 0.0"/>
             <origin xyz="${-(body_length/2) + 0.1} ${(rear_wheel_width/2 + body_width/2) * reflect} ${-(body_height/2) + 0.1}"/>
+            <limit effort="0.0" velocity="${traverse_max_speed / rear_wheel_diameter}"/> <!-- rolling axle -->
+            <!-- <limit effort="100000.00" velocity="${traverse_max_speed / rear_wheel_diameter}"/> -->
         </joint>
         <!-- The Transmission -->
@@ -200,7 +219,9 @@
             <type>transmission_interface/SimpleTransmission</type>
             <joint name="${prefix}_rear_axle">
+                <!-- <hardwareInterface>hardware_interface/VelocityJointInterface</hardwareInterface> --> <!-- rolling axle -->
                 <hardwareInterface>hardware_interface/EffortJointInterface</hardwareInterface>
             </joint>
             <actuator name="${prefix}_rear_wheel_motor">
+                <!-- <hardwareInterface>hardware_interface/VelocityJointInterface</hardwareInterface> --> <!-- rolling axle -->
                 <hardwareInterface>hardware_interface/EffortJointInterface</hardwareInterface>
                 <mechanicalReduction>1</mechanicalReduction>
@@ -217,5 +238,6 @@
     <gazebo>
         <plugin name="gazebo_ros_control" filename="libgazebo_ros_control.so">
-            <robotNamespace>/basic_laser_pig</robotNamespace>
+            <robotNamespace>/basic_pig</robotNamespace>
+            <robotSimType>gazebo_ros_control/AckermannRobotHWSim</robotSimType> <!-- THIS IS NEW -->
         </plugin>
     </gazebo>

Commit message: Laser_pig_stuff

File: urdf/basic_laser_pig.urdf.xacro (robot description, xacro)
@@ -116,4 +116,56 @@
       </inertial>
     </link>
+    <!-- IMU -->
+    <joint name="imu_joint" type="fixed">
+      <axis xyz="1 0 0 "/> <!-- 0 1 0 -->
+      <origin xyz="0 0 0.19"/>
+      <parent link ="chassis"/>
+      <child link ="imu_link"/>
+    </joint>
+    <link name="imu_link">
+	<inertial>
+	    <mass value="0.001"/>
+	    <origin rpy="0 0 0" xyz="0 0 0"/>
+	    <inertia ixx="0.0001" ixy="0" ixz="0" iyy="0.000001" iyz="0" izz="0.0001"/>
+	</inertial>
+	<visual>
+	    <origin rpy="0 0 0" xyz="0 0 0"/>
+	    <geometry>
+	      <box size="0.001 0.001 0.001"/>
+	    </geometry>
+	</visual>
+	  <collision>
+	    <origin rpy="0 0 0" xyz="0 0 0"/>
+	    <geometry>
+	      <box size=".001 .001 .001"/>
+	    </geometry>
+	  </collision>
+	</link>
+    <!-- GPS -->
+    <joint name="gps_joint" type="fixed">
+      <axis xyz="0 0 0 "/>
+      <origin xyz="0 0 0.19"/>
+      <parent link ="chassis"/>
+      <child link ="gps_link"/>
+    </joint>
+    <link name="gps_link">
+	<inertial>
+	    <mass value="0.001"/>
+	    <origin rpy="0 0 0" xyz="0 0 0"/>
+	    <inertia ixx="0.0001" ixy="0" ixz="0" iyy="0.000001" iyz="0" izz="0.0001"/>
+	</inertial>
+	<visual>
+	    <origin rpy="0 0 0" xyz="0 0 0"/>
+	    <geometry>
+	      <box size="0.001 0.001 0.001"/>
+	    </geometry>
+	</visual>
+	  <collision>
+	    <origin rpy="0 0 0" xyz="0 0 0"/>
+	    <geometry>
+	      <box size=".001 .001 .001"/>
+	    </geometry>
+	  </collision>
+	</link>
     <!-- Steering Macro -->
     <xacro:macro name="steering_link" params="prefix reflect">
@@ -167,4 +219,28 @@
                     <cylinder radius="${front_wheel_diameter/2}" length="${front_wheel_width}"/>
                 </geometry>
+		<surface>
+			<friction>
+				<torsional>
+					<coefficient>2.0</coefficient>
+					<surface_radius>.3025</surface_radius>
+					<use_patch_radius>false</use_patch_radius>
+					<ode>
+						<slip>0.5</slip>
+					</ode>
+				</torsional>
+				<ode>
+					<mu>50000.00</mu>
+					<mu2>50000.00</mu2>
+					<fdir1>1.00000 0.00000 0.00000</fdir1>
+					<slip1>0.00000</slip1>
+					<slip2>0.00000</slip2>
+				</ode>
+			</friction>
+			<contact>
+				<ode>
+					<min_depth>0.3025</min_depth>
+				</ode>
+			</contact>
+		</surface>
             </collision>
             <xacro:default_inertial mass="${front_wheel_mass}"/>
@@ -204,4 +280,28 @@
                     <cylinder radius="${rear_wheel_diameter/2}" length="${rear_wheel_width}"/>
                 </geometry>
+		<surface>
+			<friction>
+				<torsional>
+					<coefficient>2.0</coefficient>
+					<surface_radius>.3175</surface_radius>
+					<use_patch_radius>false</use_patch_radius>
+					<ode>
+						<slip>0.5</slip>
+					</ode>
+				</torsional>
+				<ode>
+					<mu>50000.00</mu>
+					<mu2>50000.00</mu2>
+					<fdir1>1.00000 0.00000 0.00000</fdir1>
+					<slip1>0.00000</slip1>
+					<slip2>0.00000</slip2>
+				</ode>
+			</friction>
+			<contact>
+				<ode>
+					<min_depth>0.3175</min_depth>
+				</ode>
+			</contact>
+		</surface>
             </collision>
             <xacro:default_inertial mass="${rear_wheel_mass}"/>
@@ -241,4 +341,25 @@
             <robotSimType>gazebo_ros_control/AckermannRobotHWSim</robotSimType> <!-- THIS IS NEW -->
         </plugin>
+        <plugin name="imu_plugin" filename="libhector_gazebo_ros_imu.so">
+            <alwaysOn>true</alwaysOn>
+            <bodyName>chassis</bodyName>
+            <topicName>imu</topicName>
+            <serviceName>imu_service</serviceName>
+            <gaussianNoise>0.0</gaussianNoise>
+            <updateRate>20.0</updateRate>
+        </plugin>
+        <plugin name="gps_plugin" filename="libhector_gazebo_ros_gps.so">
+            <alwayson>1</alwayson>
+            <updaterate>10.0</updaterate>
+            <bodyname>chassis</bodyname>
+            <topicname>fix</topicname>
+            <velocitytopicname>fix_vel</velocitytopicname>
+            <drift>5.0 5.0 5.0</drift>
+            <gaussiannoise>0.1 0.1 0.1 </gaussiannoise>
+            <velocitydrift>0 0 0</velocitydrift>
+            <velocitygaussiannoise>0.1 0.1 0.1</velocitygaussiannoise>
+            <referenceLatitude>37.634047</referenceLatitude>
+            <referenceLongitude>-97.269368</referenceLongitude>
+        </plugin>
     </gazebo>
 </robot>

Commit message: For testing Gmapping

File: urdf/basic_laser_pig.urdf.xacro (robot description, xacro)
@@ -22,9 +22,9 @@
     <xacro:property name="body_width" value="0.680618" />
     <xacro:property name="body_height" value="1.065022" />
-    <xacro:property name="body_mass" value="200.0"/>
+    <xacro:property name="body_mass" value="20.3"/>
     <!-- Front Wheel Properties -->
     <xacro:property name="front_wheel_width" value=".254" />
     <xacro:property name="front_wheel_diameter" value="0.605" />
-    <xacro:property name="front_wheel_mass" value="10"/>
+    <xacro:property name="front_wheel_mass" value="20"/>
     <!-- Steering Link Properties -->
     <xacro:property name="steering_width" value="${front_wheel_width/4}" />
@@ -34,5 +34,5 @@
     <xacro:property name="rear_wheel_width" value="${front_wheel_width+steering_width}" />
     <xacro:property name="rear_wheel_diameter" value="0.635" />
-    <xacro:property name="rear_wheel_mass" value="12"/>
+    <xacro:property name="rear_wheel_mass" value="22.8"/>
     <!-- Camera Properties -->
     <xacro:property name="camera_link" value="0.04"/>
@@ -221,28 +221,28 @@
                     <cylinder radius="${front_wheel_diameter/2}" length="0.02"/>
                 </geometry>
-                    <surface>
-                        <friction>
-                            <torsional>
-                                <coefficient>2.0</coefficient>
-                                <surface_radius>.3025</surface_radius>
-                                <use_patch_radius>false</use_patch_radius>
-                                <ode>
-                                    <slip>0.5</slip>
-                                </ode>
-                            </torsional>
+                <surface>
+                    <friction>
+                        <torsional>
+                            <coefficient>2.0</coefficient>
+                            <surface_radius>.3025</surface_radius>
+                            <use_patch_radius>false</use_patch_radius>
                             <ode>
-                                <mu>50000.00</mu>
-                                <mu2>50000.00</mu2>
-                                <fdir1>1.00000 0.00000 0.00000</fdir1>
-                                <slip1>0.00000</slip1>
-                                <slip2>0.00000</slip2>
+                                <slip>0.0</slip>
                             </ode>
-                        </friction>
-                        <contact>
-                            <ode>
-                                <min_depth>0.03</min_depth>
-                            </ode>
-                        </contact>
-                    </surface>
+                        </torsional>
+                        <ode>
+                            <mu>70000.00</mu>
+                            <mu2>70000.00</mu2>
+                            <fdir1>1.00000 0.00000 0.00000</fdir1>
+                            <slip1>0.00000</slip1>
+                            <slip2>0.00000</slip2>
+                        </ode>
+                    </friction>
+                    <contact>
+                        <ode>
+                            <min_depth>0.4025</min_depth>
+                        </ode>
+                    </contact>
+                </surface>
             </collision>
             <xacro:default_inertial mass="${front_wheel_mass}"/>
@@ -309,5 +309,5 @@
                 <origin xyz="0.0 0.0 0.0" rpy="${degrees_90} 0.0 0.0"/>
                 <geometry>
-                    <cylinder radius="${rear_wheel_diameter/2}" length="0.02"/>
+                    <cylinder radius="${rear_wheel_diameter/2}" length="0.01"/>
                 </geometry>
             </collision>
@@ -365,23 +365,28 @@
         <plugin name="imu_plugin" filename="libhector_gazebo_ros_imu.so">
             <alwaysOn>true</alwaysOn>
-            <bodyName>chassis</bodyName>
-            <topicName>imu/data</topicName>
-            <serviceName>imu/is_calibrated</serviceName>
+            <bodyName>imu_link</bodyName>
+            <topicName>imu/data</topicName> <!-- Lets solve the namepsace issues -->
+            <accelDrift>0.005 0.005 0.005</accelDrift>
+            <accelGaussianNoise>0.005 0.005 0.005</accelGaussianNoise>
+            <rateDrift>0.005 0.005 0.005</rateDrift>
+            <rateGaussianNoise>0.005 0.005 0.005</rateGaussianNoise>
+            <headingDrift>0.005 0.005 0.005</headingDrift>
             <gaussianNoise>0.0</gaussianNoise>
-            <updateRate>20.0</updateRate>
+            <updateRate>50.0</updateRate>
             <xyzOffsets>0 0 0</xyzOffsets>
             <rpyOffsets>0 0 0</rpyOffsets>
         </plugin>
         <plugin name="gps_plugin" filename="libhector_gazebo_ros_gps.so">
-            <alwayson>1</alwayson>
-            <updaterate>10.0</updaterate>
-            <bodyname>chassis</bodyname>
-            <topicname>fix</topicname>
-            <velocitytopicname>fix_vel</velocitytopicname>
-            <gaussiannoise>0.1 0.1 0.1 </gaussiannoise>
-            <velocitydrift>0 0 0</velocitydrift>
-            <velocitygaussiannoise>0.1 0.1 0.1</velocitygaussiannoise>
+            <alwaysOn>1</alwaysOn>
+            <updateRate>40.0</updateRate>
+            <frameId>base_link</frameId> <!-- Defaults to world? don't put in a "/"-->
+            <bodyName>chassis</bodyName>
+            <topicName>fix</topicName>
+            <velocityTopicName>fix_vel</velocityTopicName>
+            <drift>0.0001 0.0001 0.0001</drift>
             <referenceLatitude>37.634047</referenceLatitude>
             <referenceLongitude>-97.269368</referenceLongitude>
+            <referenceHeading>0</referenceHeading>
+            <referenceAltitude>0</referenceAltitude>
         </plugin>
     </gazebo>
