Commit message: Proper Description

File: urdf/basic_laser_pig.urdf.xacro (robot description, xacro)
@@ -66,5 +66,5 @@
     <joint name="laser_link_joint" type="fixed">
       <axis xyz="0 0 0" />
-      <origin xyz="${(body_length) + 0.1} 0.0 0.0" rpy="0 0 0"/>
+      <origin xyz="${(body_length) + 0.1} 0.0 0.0" rpy="0 0 ${degrees_180}"/> <!-- Was reversed in real world -->
       <parent link="chassis"/>
       <child link="laser_link"/>
@@ -350,4 +350,80 @@
         </transmission>
     </xacro:macro>
+    <!-- Ackermann Steering Macro, this is a dummy joint so it has no visual  -->
+    <xacro:macro name="ackermann_steering_link">
+        <link name="ackermann_steering_link">
+            <!-- <visual>
+                <origin xyz="0.0 0.0 0.0" rpy="${degrees_90} 0.0 0.0"/>
+                <geometry>
+                    <cylinder radius="${steering_diameter}" length="${steering_width}"/>
+                </geometry>
+            </visual> -->
+            <collision>
+                <origin xyz="0.0 0.0 0.0" rpy="${degrees_90} 0.0 0.0"/>
+                <geometry>
+                    <cylinder radius="${steering_diameter}" length="${steering_width}"/>
+                </geometry>
+            </collision>
+            <xacro:default_inertial mass="${steering_mass}"/>
+        </link>
+        <joint name="ackermann_steering_joint" type="revolute">
+            <parent link="chassis"/>
+            <child link="ackermann_steering_link"/>
+            <axis xyz="0.0 0.0 0.1"/>
+            <origin xyz="${(body_length)- 0.2} 0.0 1.0" rpy="0.0 0.0 0.0"/>
+            <limit lower="${steering_min_angle}" upper="${steering_max_angle}" effort="100000.00" velocity="${steering_speed}"/>
+            <!-- effort needs to be very high so we are not constrained by the environment-->
+        </joint>
+        <!-- The Transmission -->
+        <transmission name="ackermann_steering_link_trans">
+            <type>transmission_interface/SimpleTransmission</type>
+            <joint name="ackermann_steering_joint">
+                <hardwareInterface>hardware_interface/PositionJointInterface</hardwareInterface>
+            </joint>
+            <actuator name="ackermann_steering_link_motor">
+                <hardwareInterface>hardware_interface/PositionJointInterface</hardwareInterface>
+                <mechanicalReduction>1</mechanicalReduction>
+            </actuator>
+        </transmission>
+    </xacro:macro>
+    <!-- Ackermann Wheel Macro, this is a dummy joint so it has no visual -->
+    <xacro:macro name="ackermann_wheel_link">
+        <link name="ackermann_rear_wheel">
+            <!-- <visual>
+                <origin xyz="0.0 0.0 0.0" rpy="${degrees_90} 0.0 0.0"/>
+                <geometry>
+                    <cylinder radius="${front_wheel_diameter/2}" length="${front_wheel_width}"/>
+                </geometry>
+            </visual> -->
+            <collision>
+                <origin xyz="0.0 0.0 0.0" rpy="${degrees_90} 0.0 0.0"/>
+                <geometry>
+                    <cylinder radius="${front_wheel_diameter/2}" length="0.01"/>
+                </geometry>
+            </collision>
+            <xacro:default_inertial mass="${steering_mass}"/>
+        </link>
+        <joint name="ackermann_rear_axle" type="continuous">
+            <parent link="chassis"/>
+            <child link="ackermann_rear_wheel"/>
+            <axis xyz="0.0 0.1 0.0"/>
+            <origin xyz="0.0 0.0 1.0" rpy="0.0 0.0 0.0"/>
+            <!-- <limit effort="0.0" velocity="${traverse_max_speed / rear_wheel_diameter}"/> --> <!-- rolling axle -->
+            <!-- <limit effort="100000.00" velocity="${traverse_max_speed / rear_wheel_diameter}"/> -->
+        </joint>
+        <!-- The Transmission -->
+        <transmission name="ackermann_rear_wheel_trans">
+            <type>transmission_interface/SimpleTransmission</type>
+            <joint name="ackermann_rear_axle">
+                <!-- <hardwareInterface>hardware_interface/VelocityJointInterface</hardwareInterface> --> <!-- rolling axle -->
+                <hardwareInterface>hardware_interface/EffortJointInterface</hardwareInterface>
+            </joint>
+            <actuator name="ackermann_rear_wheel_motor">
+                <!-- <hardwareInterface>hardware_interface/VelocityJointInterface</hardwareInterface> --> <!-- rolling axle -->
+                <hardwareInterface>hardware_interface/EffortJointInterface</hardwareInterface>
+                <mechanicalReduction>1</mechanicalReduction>
+            </actuator>
+        </transmission>
+    </xacro:macro>
     <xacro:steering_link prefix="left" reflect="1" />
     <xacro:steering_link prefix="right" reflect="-1" />
@@ -358,4 +434,6 @@
     <xacro:rear_wheel_link prefix="left" reflect="1" />
     <xacro:rear_wheel_link prefix="right" reflect="-1" />
+    <xacro:ackermann_steering_link />
+    <xacro:ackermann_wheel_link />
     <!-- Gazebo plugin for ROS Control -->
     <gazebo>

Commit message: Description Changes

File: urdf/basic_laser_pig.urdf.xacro (robot description, xacro)
@@ -8,6 +8,6 @@
     <!-- vehiclur velocity properties -->
     <xacro:property name="steering_speed" value="1.0472"/> <!-- units of rad/s -->
-    <xacro:property name="steering_max_angle" value="${degrees_30}"/> <!-- units of rad -->
-    <xacro:property name="steering_min_angle" value="-${degrees_30}"/> <!-- units of rad -->
+    <xacro:property name="steering_max_angle" value="${degrees_45}"/> <!-- units of rad, used to be 0.523 -->
+    <xacro:property name="steering_min_angle" value="-${degrees_45}"/> <!-- units of rad, used to be 0.523 -->
     <xacro:property name="traverse_max_speed" value="4.785"/> <!-- units of m/s 4.785-->
     <!-- Inertia Generator -->
@@ -25,5 +25,5 @@
     <!-- Front Wheel Properties -->
     <xacro:property name="front_wheel_width" value=".254" />
-    <xacro:property name="front_wheel_diameter" value="0.605" />
+    <xacro:property name="front_wheel_diameter" value="0.572" />
     <xacro:property name="front_wheel_mass" value="20"/>
     <!-- Steering Link Properties -->

Commit message: Dual Laser

File: urdf/basic_laser_pig.urdf.xacro (robot description, xacro)
@@ -66,5 +66,5 @@
     <joint name="laser_link_joint" type="fixed">
       <axis xyz="0 0 0" />
-      <origin xyz="${(body_length) + 0.1} 0.0 0.0" rpy="0 0 ${degrees_180}"/> <!-- Was reversed in real world -->
+      <origin xyz="${(body_length) + 0.1} 0.0 0.0" rpy="0 0 0"/> <!-- Was reversed in real world -->
       <parent link="chassis"/>
       <child link="laser_link"/>
@@ -72,4 +72,30 @@
      <!-- Laser -->
     <link name="laser_link">
+      <collision>
+        <origin xyz="0 0 0" rpy="0 0 0"/>
+        <geometry>
+          <cylinder radius=".05" length="0.04"/>
+        </geometry>
+      </collision>
+      <visual>
+        <origin xyz="0 0 0" rpy="0 0 0"/>
+        <geometry>
+          <cylinder radius=".05" length="0.04"/>
+        </geometry>
+      </visual>
+      <inertial>
+        <mass value="1e-5" />
+        <origin xyz="0 0 0" rpy="0 0 0"/>
+        <inertia ixx="1e-6" ixy="0" ixz="0" iyy="1e-6" iyz="0" izz="1e-6" />
+      </inertial>
+    </link>
+    <!-- Laser link -->
+    <joint name="laser_link_joint_back" type="fixed">
+      <axis xyz="0 0 0" />
+      <origin xyz="-0.15 0.0 0.0" rpy="0 0 ${degrees_180}"/> <!-- Was reversed in real world -->
+      <parent link="chassis"/>
+      <child link="laser_link_back"/>
+    </joint>
+    <link name="laser_link_back">
       <collision>
         <origin xyz="0 0 0" rpy="0 0 0"/>
