Commit message: Fixing Fils

File: urdf/basic_laser_pig.urdf.xacro (robot description, xacro)
@@ -1,5 +1,6 @@
 <?xml version="1.0"?>
-<robot xmlns:xacro="http://www.ros.org/wiki/xacro" name="basic_pig">
+<robot xmlns:xacro="http://www.ros.org/wiki/xacro" name="basic_laser_pig">
     <!-- Degree-to-radian conversions -->
+    <xacro:property name="degrees_30" value="0.523598776"/>
     <xacro:property name="degrees_45" value="0.785398163"/>
     <xacro:property name="degrees_90" value="1.57079633"/>
@@ -7,7 +8,7 @@
     <!-- vehiclur velocity properties -->
     <xacro:property name="steering_speed" value="1.0472"/> <!-- units of rad/s -->
-    <xacro:property name="steering_max_angle" value="0.3"/> <!-- units of rad -->
-    <xacro:property name="steering_min_angle" value="-0.3"/> <!-- units of rad -->
-    <xacro:property name="traverse_max_speed" value="4.785"/> <!-- units of m/s -->
+    <xacro:property name="steering_max_angle" value="${degrees_45}"/> <!-- units of rad, used to be 0.523 -->
+    <xacro:property name="steering_min_angle" value="-${degrees_45}"/> <!-- units of rad, used to be 0.523 -->
+    <xacro:property name="traverse_max_speed" value="4.785"/> <!-- units of m/s 4.785-->
     <!-- Inertia Generator -->
     <xacro:macro name="default_inertial" params="mass">
@@ -24,5 +25,5 @@
     <!-- Front Wheel Properties -->
     <xacro:property name="front_wheel_width" value=".254" />
-    <xacro:property name="front_wheel_diameter" value="0.605" />
+    <xacro:property name="front_wheel_diameter" value="0.572" />
     <xacro:property name="front_wheel_mass" value="20"/>
     <!-- Steering Link Properties -->
@@ -43,5 +44,5 @@
     <link name="chassis">
         <visual>
-            <origin xyz="0.0 0.0 0.0" rpy="0.0 0.0 0.0"/>
+            <origin xyz="${(body_length/2) - 0.1} 0.0 0.0" rpy="0.0 0.0 0.0"/>
             <geometry>
                 <box size="${body_length} ${body_width} ${body_height}"/>
@@ -50,5 +51,5 @@
         </visual>
         <collision>
-            <origin xyz="0.0 0.0 0.0" rpy="0.0 0.0 0.0"/>
+            <origin xyz="${(body_length/2) - 0.1} 0.0 0.0" rpy="0.0 0.0 0.0"/>
             <geometry>
                 <box size="${body_length} ${body_width} ${body_height}"/>
@@ -65,5 +66,5 @@
     <joint name="laser_link_joint" type="fixed">
       <axis xyz="0 0 0" />
-      <origin xyz="${(body_length/2) - 0.1} 0.0 ${(body_height/2 + 0.1)}" rpy="0 0 0"/>
+      <origin xyz="${(body_length) + 0.1} 0.0 0.0" rpy="0 0 0"/> <!-- Was reversed in real world -->
       <parent link="chassis"/>
       <child link="laser_link"/>
@@ -92,5 +93,5 @@
     <joint name="camera_link_joint" type="fixed">
       <axis xyz="0 1 0" />
-      <origin xyz="${(body_length/2) - 0.1} 0.0 ${(body_height/2 + 0.2)}" rpy="0 0 0"/>
+      <origin xyz="${(body_length) - 0.1} 0.0 ${(body_height/2 + 0.2)}" rpy="0 0 0"/>
       <parent link="chassis"/>
       <child link="camera_link"/>
@@ -100,5 +101,5 @@
         <origin xyz="0 0 0" rpy="0 0 0"/>
         <geometry>
-      <box size="${camera_link} ${camera_link} ${camera_link}"/>
+        <box size="${camera_link} ${camera_link} ${camera_link}"/>
         </geometry>
       </collision>
@@ -106,5 +107,5 @@
         <origin xyz="0 0 0" rpy="0 0 0"/>
         <geometry>
-      <box size="${camera_link} ${camera_link} ${camera_link}"/>
+        <box size="${camera_link} ${camera_link} ${camera_link}"/>
         </geometry>
         <material name="red"/>
@@ -118,29 +119,29 @@
     <!-- IMU -->
     <joint name="imu_joint" type="fixed">
-      <axis xyz="1 0 0 "/> <!-- 0 1 0 -->
-      <origin xyz="0 0 0.19"/>
-      <parent link ="chassis"/>
-      <child link ="imu_link"/>
+        <axis xyz="1 0 0 "/> <!-- 0 1 0 -->
+        <origin xyz="0 0 0.19"/>
+        <parent link ="chassis"/>
+        <child link ="imu_link"/>
     </joint>
     <link name="imu_link">
-	<inertial>
-	    <mass value="0.001"/>
-	    <origin rpy="0 0 0" xyz="0 0 0"/>
-	    <inertia ixx="0.0001" ixy="0" ixz="0" iyy="0.000001" iyz="0" izz="0.0001"/>
-	</inertial>
-	<visual>
-	    <origin rpy="0 0 0" xyz="0 0 0"/>
-	    <geometry>
-	      <box size="0.001 0.001 0.001"/>
-	    </geometry>
-	</visual>
-	  <collision>
-	    <origin rpy="0 0 0" xyz="0 0 0"/>
-	    <geometry>
-	      <box size=".001 .001 .001"/>
-	    </geometry>
-	  </collision>
+        <inertial>
+            <mass value="0.001"/>
+            <origin rpy="0 0 0" xyz="0 0 0"/>
+            <inertia ixx="0.0001" ixy="0" ixz="0" iyy="0.000001" iyz="0" izz="0.0001"/>
+        </inertial>
+        <visual>
+            <origin rpy="0 0 0" xyz="0 0 0"/>
+            <geometry>
+            <box size="0.001 0.001 0.001"/>
+            </geometry>
+        </visual>
+        <collision>
+            <origin rpy="0 0 0" xyz="0 0 0"/>
+            <geometry>
+            <box size=".001 .001 .001"/>
+            </geometry>
+        </collision>
 	</link>
-    <!-- GPS -->
+    <!-- GPS (THIS JOINT IS UNNECESSARY)
     <joint name="gps_joint" type="fixed">
       <axis xyz="0 0 0 "/>
@@ -150,22 +151,23 @@
     </joint>
     <link name="gps_link">
-	<inertial>
-	    <mass value="0.001"/>
-	    <origin rpy="0 0 0" xyz="0 0 0"/>
-	    <inertia ixx="0.0001" ixy="0" ixz="0" iyy="0.000001" iyz="0" izz="0.0001"/>
-	</inertial>
-	<visual>
-	    <origin rpy="0 0 0" xyz="0 0 0"/>
-	    <geometry>
-	      <box size="0.001 0.001 0.001"/>
-	    </geometry>
-	</visual>
-	  <collision>
-	    <origin rpy="0 0 0" xyz="0 0 0"/>
-	    <geometry>
-	      <box size=".001 .001 .001"/>
-	    </geometry>
-	  </collision>
+        <inertial>
+            <mass value="0.001"/>
+            <origin rpy="0 0 0" xyz="0 0 0"/>
+            <inertia ixx="0.0001" ixy="0" ixz="0" iyy="0.000001" iyz="0" izz="0.0001"/>
+        </inertial>
+        <visual>
+            <origin rpy="0 0 0" xyz="0 0 0"/>
+            <geometry>
+            <box size="0.001 0.001 0.001"/>
+            </geometry>
+        </visual>
+        <collision>
+            <origin rpy="0 0 0" xyz="0 0 0"/>
+            <geometry>
+            <box size=".001 .001 .001"/>
+            </geometry>
+        </collision>
 	</link>
+    -->
     <!-- Steering Macro -->
     <xacro:macro name="steering_link" params="prefix reflect">
@@ -189,5 +191,5 @@
             <child link="${prefix}_steering_link"/>
             <axis xyz="0.0 0.0 0.1"/>
-            <origin xyz="${(body_length / 2)- 0.1} ${(body_width / 2 + steering_width / 2) * reflect} ${-(body_height/2) + 0.1}" rpy="0.0 0.0 0.0"/>
+            <origin xyz="${(body_length)- 0.2} ${(body_width / 2 + steering_width / 2 + 0.1) * reflect} ${-(body_height/2) + 0.1}" rpy="0.0 0.0 0.0"/>
             <limit lower="${steering_min_angle}" upper="${steering_max_angle}" effort="100000.00" velocity="${steering_speed}"/>
             <!-- effort needs to be very high so we are not constrained by the environment-->
@@ -217,30 +219,30 @@
                 <origin xyz="0.0 0.0 0.0" rpy="${degrees_90} 0.0 0.0"/>
                 <geometry>
-                    <cylinder radius="${front_wheel_diameter/2}" length="${front_wheel_width}"/>
-                </geometry>
-		<surface>
-			<friction>
-				<torsional>
-					<coefficient>2.0</coefficient>
-					<surface_radius>.3025</surface_radius>
-					<use_patch_radius>false</use_patch_radius>
-					<ode>
-						<slip>0.5</slip>
-					</ode>
-				</torsional>
-				<ode>
-					<mu>50000.00</mu>
-					<mu2>50000.00</mu2>
-					<fdir1>1.00000 0.00000 0.00000</fdir1>
-					<slip1>0.00000</slip1>
-					<slip2>0.00000</slip2>
-				</ode>
-			</friction>
-			<contact>
-				<ode>
-					<min_depth>0.3025</min_depth>
-				</ode>
-			</contact>
-		</surface>
+                    <cylinder radius="${front_wheel_diameter/2}" length="0.02"/>
+                </geometry>
+                <surface>
+                    <friction>
+                        <torsional>
+                            <coefficient>2.0</coefficient>
+                            <surface_radius>.3025</surface_radius>
+                            <use_patch_radius>false</use_patch_radius>
+                            <ode>
+                                <slip>0.0</slip>
+                            </ode>
+                        </torsional>
+                        <ode>
+                            <mu>70000.00</mu>
+                            <mu2>70000.00</mu2>
+                            <fdir1>1.00000 0.00000 0.00000</fdir1>
+                            <slip1>0.00000</slip1>
+                            <slip2>0.00000</slip2>
+                        </ode>
+                    </friction>
+                    <contact>
+                        <ode>
+                            <min_depth>0.4025</min_depth>
+                        </ode>
+                    </contact>
+                </surface>
             </collision>
             <xacro:default_inertial mass="${front_wheel_mass}"/>
@@ -266,4 +268,33 @@
         </transmission>
     </xacro:macro>
+    <!-- Rear Wheel Prismatic Link Macro -->
+    <xacro:macro name="rear_wheel_strut_link" params="prefix reflect">
+        <link name="${prefix}_rear_wheel_strut">
+            <visual>
+                <origin xyz="0.0 0.0 0.0" rpy="${degrees_90} 0.0 0.0"/>
+                <geometry>
+                    <cylinder radius="0.1" length="0.02"/>
+                </geometry>
+            </visual>
+            <collision>
+                <origin xyz="0.0 0.0 0.0" rpy="${degrees_90} 0.0 0.0"/>
+                <geometry>
+                    <cylinder radius="0.1" length="0.02"/>
+                </geometry>
+            </collision>
+            <xacro:default_inertial mass="${rear_wheel_mass}"/>
+        </link>
+        <joint name="${prefix}_rear_strut}" type="prismatic">
+            <parent link="chassis"/>
+            <child link="${prefix}_rear_wheel_strut"/>
+            <axis xyz="0.0 0.0 0.1"/>
+            <origin xyz="0.0 ${(body_width/2 + 0.1) * reflect} ${-(body_height/2) + 0.1}"/>
+            <limit lower="-0.05" upper="0.05" effort="1000.0" velocity="1.0"/>
+            <dynamics damping="2.0" friction="8000.0"/>
+        </joint>
+        <gazebo reference="${prefix}_rear_strut}">
+            <implicitSpringDamper>true</implicitSpringDamper>
+        </gazebo>
+    </xacro:macro>
     <!-- Rear Wheel Macro -->
     <xacro:macro name="rear_wheel_link" params="prefix reflect">
@@ -278,39 +309,29 @@
                 <origin xyz="0.0 0.0 0.0" rpy="${degrees_90} 0.0 0.0"/>
                 <geometry>
-                    <cylinder radius="${rear_wheel_diameter/2}" length="${rear_wheel_width}"/>
-                </geometry>
-		<surface>
-			<friction>
-				<torsional>
-					<coefficient>2.0</coefficient>
-					<surface_radius>.3175</surface_radius>
-					<use_patch_radius>false</use_patch_radius>
-					<ode>
-						<slip>0.5</slip>
-					</ode>
-				</torsional>
-				<ode>
-					<mu>50000.00</mu>
-					<mu2>50000.00</mu2>
-					<fdir1>1.00000 0.00000 0.00000</fdir1>
-					<slip1>0.00000</slip1>
-					<slip2>0.00000</slip2>
-				</ode>
-			</friction>
-			<contact>
-				<ode>
-					<min_depth>0.3175</min_depth>
-				</ode>
-			</contact>
-		</surface>
-            </collision>
+                    <cylinder radius="${rear_wheel_diameter/2}" length="0.01"/>
+                </geometry>
+            </collision>
+            <surface>
+                <contact>
+                    <ode>
+                        <min_depth>0.01</min_depth>
+                    </ode>
+                </contact>
+                <friction>
+                    <ode>
+                        <mu>1</mu>
+                        <mu2>1</mu2>
+                        <fdir1>1.0 0 0</fdir1>
+                    </ode>
+                </friction>
+            </surface>
             <xacro:default_inertial mass="${rear_wheel_mass}"/>
         </link>
         <joint name="${prefix}_rear_axle" type="continuous">
-            <parent link="chassis"/>
+            <parent link="${prefix}_rear_wheel_strut"/>
             <child link="${prefix}_rear_wheel"/>
             <axis xyz="0.0 0.1 0.0"/>
-            <origin xyz="${-(body_length/2) + 0.1} ${(rear_wheel_width/2 + body_width/2) * reflect} ${-(body_height/2) + 0.1}"/>
-            <limit effort="0.0" velocity="${traverse_max_speed / rear_wheel_diameter}"/> <!-- rolling axle -->
+            <origin xyz="0.0 ${(rear_wheel_width/2) * reflect} 0.0"/>
+            <!-- <limit effort="0.0" velocity="${traverse_max_speed / rear_wheel_diameter}"/> --> <!-- rolling axle -->
             <!-- <limit effort="100000.00" velocity="${traverse_max_speed / rear_wheel_diameter}"/> -->
         </joint>
@@ -329,36 +350,121 @@
         </transmission>
     </xacro:macro>
+    <!-- Ackermann Steering Macro, this is a dummy joint so it has no visual  -->
+    <xacro:macro name="ackermann_steering_link">
+        <link name="ackermann_steering_link">
+            <!-- <visual>
+                <origin xyz="0.0 0.0 0.0" rpy="${degrees_90} 0.0 0.0"/>
+                <geometry>
+                    <cylinder radius="${steering_diameter}" length="${steering_width}"/>
+                </geometry>
+            </visual> -->
+            <collision>
+                <origin xyz="0.0 0.0 0.0" rpy="${degrees_90} 0.0 0.0"/>
+                <geometry>
+                    <cylinder radius="${steering_diameter}" length="${steering_width}"/>
+                </geometry>
+            </collision>
+            <xacro:default_inertial mass="${steering_mass}"/>
+        </link>
+        <joint name="ackermann_steering_joint" type="revolute">
+            <parent link="chassis"/>
+            <child link="ackermann_steering_link"/>
+            <axis xyz="0.0 0.0 0.1"/>
+            <origin xyz="${(body_length)- 0.2} 0.0 1.0" rpy="0.0 0.0 0.0"/>
+            <limit lower="${steering_min_angle}" upper="${steering_max_angle}" effort="100000.00" velocity="${steering_speed}"/>
+            <!-- effort needs to be very high so we are not constrained by the environment-->
+        </joint>
+        <!-- The Transmission -->
+        <transmission name="ackermann_steering_link_trans">
+            <type>transmission_interface/SimpleTransmission</type>
+            <joint name="ackermann_steering_joint">
+                <hardwareInterface>hardware_interface/PositionJointInterface</hardwareInterface>
+            </joint>
+            <actuator name="ackermann_steering_link_motor">
+                <hardwareInterface>hardware_interface/PositionJointInterface</hardwareInterface>
+                <mechanicalReduction>1</mechanicalReduction>
+            </actuator>
+        </transmission>
+    </xacro:macro>
+    <!-- Ackermann Wheel Macro, this is a dummy joint so it has no visual -->
+    <xacro:macro name="ackermann_wheel_link">
+        <link name="ackermann_rear_wheel">
+            <!-- <visual>
+                <origin xyz="0.0 0.0 0.0" rpy="${degrees_90} 0.0 0.0"/>
+                <geometry>
+                    <cylinder radius="${front_wheel_diameter/2}" length="${front_wheel_width}"/>
+                </geometry>
+            </visual> -->
+            <collision>
+                <origin xyz="0.0 0.0 0.0" rpy="${degrees_90} 0.0 0.0"/>
+                <geometry>
+                    <cylinder radius="${front_wheel_diameter/2}" length="0.01"/>
+                </geometry>
+            </collision>
+            <xacro:default_inertial mass="${steering_mass}"/>
+        </link>
+        <joint name="ackermann_rear_axle" type="continuous">
+            <parent link="chassis"/>
+            <child link="ackermann_rear_wheel"/>
+            <axis xyz="0.0 0.1 0.0"/>
+            <origin xyz="0.0 0.0 1.0" rpy="0.0 0.0 0.0"/>
+            <!-- <limit effort="0.0" velocity="${traverse_max_speed / rear_wheel_diameter}"/> --> <!-- rolling axle -->
+            <!-- <limit effort="100000.00" velocity="${traverse_max_speed / rear_wheel_diameter}"/> -->
+        </joint>
+        <!-- The Transmission -->
+        <transmission name="ackermann_rear_wheel_trans">
+            <type>transmission_interface/SimpleTransmission</type>
+            <joint name="ackermann_rear_axle">
+                <!-- <hardwareInterface>hardware_interface/VelocityJointInterface</hardwareInterface> --> <!-- rolling axle -->
+                <hardwareInterface>hardware_interface/EffortJointInterface</hardwareInterface>
+            </joint>
+            <actuator name="ackermann_rear_wheel_motor">
+                <!-- <hardwareInterface>hardware_interface/VelocityJointInterface</hardwareInterface> --> <!-- rolling axle -->
+                <hardwareInterface>hardware_interface/EffortJointInterface</hardwareInterface>
+                <mechanicalReduction>1</mechanicalReduction>
+            </actuator>
+        </transmission>
+    </xacro:macro>
     <xacro:steering_link prefix="left" reflect="1" />
     <xacro:steering_link prefix="right" reflect="-1" />
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
Commit message: Everything on PIG

File: urdf/basic_laser_pig.urdf.xacro (robot description, xacro)
@@ -8,6 +8,6 @@
     <!-- vehiclur velocity properties -->
     <xacro:property name="steering_speed" value="1.0472"/> <!-- units of rad/s -->
-    <xacro:property name="steering_max_angle" value="${degrees_45}"/> <!-- units of rad, used to be 0.523 -->
-    <xacro:property name="steering_min_angle" value="-${degrees_45}"/> <!-- units of rad, used to be 0.523 -->
+    <xacro:property name="steering_max_angle" value="${degrees_30}"/> <!-- units of rad, used to be 0.523 -->
+    <xacro:property name="steering_min_angle" value="-${degrees_30}"/> <!-- units of rad, used to be 0.523 -->
     <xacro:property name="traverse_max_speed" value="4.785"/> <!-- units of m/s 4.785-->
     <!-- Inertia Generator -->
@@ -63,13 +63,38 @@
         <child link="chassis" />
     </joint>
-    <!-- Laser link -->
-    <joint name="laser_link_joint" type="fixed">
+    <!-- Front Laser -->
+    <joint name="front_laser_joint" type="fixed">
       <axis xyz="0 0 0" />
-      <origin xyz="${(body_length) + 0.1} 0.0 0.0" rpy="0 0 0"/> <!-- Was reversed in real world -->
+      <origin xyz="${(body_length) + 0.1} 0.0 0.0" rpy="0 0 ${degrees_180}"/> <!-- Was reversed in real world -->
       <parent link="chassis"/>
-      <child link="laser_link"/>
-    </joint>
-     <!-- Laser -->
-    <link name="laser_link">
+      <child link="front_laser_link"/>
+    </joint>
+    <link name="front_laser_link">
+      <collision>
+        <origin xyz="0 0 0" rpy="0 0 0"/>
+        <geometry>
+          <cylinder radius=".05" length="0.04"/>
+        </geometry>
+      </collision>
+      <visual>
+        <origin xyz="0 0 0" rpy="0 0 0"/>
+        <geometry>
+          <cylinder radius=".05" length="0.04"/>
+        </geometry>
+      </visual>
+      <inertial>
+        <mass value="1e-5" />
+        <origin xyz="0 0 0" rpy="0 0 0"/>
+        <inertia ixx="1e-6" ixy="0" ixz="0" iyy="1e-6" iyz="0" izz="1e-6" />
+      </inertial>
+    </link>
+    <!-- Rear Laser -->
+    <joint name="rear_laser_joint" type="fixed">
+      <axis xyz="0 0 0" />
+      <origin xyz="-0.15 0.0 0.0" rpy="0 0 ${degrees_180}"/> <!-- Was reversed in real world -->
+      <parent link="chassis"/>
+      <child link="rear_laser_link"/>
+    </joint>
+    <link name="rear_laser_link">
       <collision>
         <origin xyz="0 0 0" rpy="0 0 0"/>
@@ -365,5 +390,5 @@
                 </geometry>
             </collision>
-            <xacro:default_inertial mass="${steering_mass}"/>
+            <xacro:default_inertial mass="0.001"/>
         </link>
         <joint name="ackermann_steering_joint" type="revolute">
@@ -402,5 +427,5 @@
                 </geometry>
             </collision>
-            <xacro:default_inertial mass="${steering_mass}"/>
+            <xacro:default_inertial mass="0.001"/>
         </link>
         <joint name="ackermann_rear_axle" type="continuous">
@@ -444,5 +469,5 @@
             <alwaysOn>true</alwaysOn>
             <bodyName>imu_link</bodyName>
-            <topicName>imu/data</topicName> <!-- Lets solve the namepsace issues -->
+            <topicName>IMU/data</topicName> <!-- Lets solve the namepsace issues -->
             <accelDrift>0.005 0.005 0.005</accelDrift>
             <accelGaussianNoise>0.005 0.005 0.005</accelGaussianNoise>
@@ -460,6 +485,6 @@
             <frameId>base_link</frameId> <!-- Defaults to world? don't put in a "/"-->
             <bodyName>chassis</bodyName>
-            <topicName>fix</topicName>
-            <velocityTopicName>fix_vel</velocityTopicName>
+            <topicName>GPS/fix</topicName>
+            <velocityTopicName>GPS/fix_vel</velocityTopicName>
             <drift>0.0001 0.0001 0.0001</drift>
             <referenceLatitude>37.634047</referenceLatitude>

Commit message: Cleaning comments

File: urdf/basic_laser_pig.urdf.xacro (robot description, xacro)
@@ -8,6 +8,6 @@
     <!-- vehiclur velocity properties -->
     <xacro:property name="steering_speed" value="1.0472"/> <!-- units of rad/s -->
-    <xacro:property name="steering_max_angle" value="${degrees_30}"/> <!-- units of rad, used to be 0.523 -->
-    <xacro:property name="steering_min_angle" value="-${degrees_30}"/> <!-- units of rad, used to be 0.523 -->
+    <xacro:property name="steering_max_angle" value="1.0"/> <!-- units of rad, needs to be 30 degreees -->
+    <xacro:property name="steering_min_angle" value="-1.0"/> <!-- units of rad, needs to be 30 degrees -->
     <xacro:property name="traverse_max_speed" value="4.785"/> <!-- units of m/s 4.785-->
     <!-- Inertia Generator -->
