Commit message: Initial changes for new model

File: urdf/little_pig_base.urdf.xacro (robot description, xacro)
@@ -1,4 +1,9 @@
 <?xml version="1.0"?>
 <robot xmlns:xacro="http://www.ros.org/wiki/xacro" name="little_pig">
+    <!-- Degree-to-radian conversions -->
+    <xacro:property name="degrees_30" value="0.523598776"/>
+    <xacro:property name="degrees_45" value="0.785398163"/>
+    <xacro:property name="degrees_90" value="1.57079633"/>
+    <xacro:property name="degrees_180" value="3.14159265"/>
     <xacro:include filename="$(find little_pig_description)/xacro/params/color_properties.xacro"/>
     <xacro:include filename="$(find little_pig_description)/xacro/params/characteristics.xacro"/>
@@ -41,3 +46,9 @@
     <xacro:rear_wheel prefix="left" reflect="1" />
     <xacro:rear_wheel prefix="right" reflect="-1" />
+    <!-- Gazebo plugin for ROS Control -->
+    <gazebo>
+        <plugin name="gazebo_ros_control" filename="libgazebo_ros_control.so">
+            <robotSimType>gazebo_ros_control/AckermannRobotHWSim</robotSimType>
+        </plugin>
+    </gazebo>
 </robot>

File: xacro/macros/_front_wheel.urdf.xacro (robot description, xacro)
@@ -8,11 +8,12 @@
                     <mesh filename="package://little_pig_description/meshes/little_pig_wheel.stl" scale="0.0254 0.0254 0.0254"/>
                 </geometry>
-                <origin rpy="0 0.0 ${1.57075 * reflect}" xyz="0 0 0.0"/>
+                <origin rpy="0.0 0.0 ${degrees_90 * reflect}" xyz="0 0 0.0"/>
                 <material name="black"/>
             </visual>
             <collision>
-                <origin xyz="0.0 0.0 0.0" rpy="0.0 0.0 ${1.57075 * reflect}"/>
+                <origin xyz="0.0 0.0 0.0" rpy="${degrees_90 * reflect} 0.0 0.0"/>
                 <geometry>
-                    <mesh filename="package://little_pig_description/meshes/little_pig_wheel.stl" scale="0.0254 0.0254 0.0254"/>
+                    <cylinder radius="${front_wheel_diameter/2}" length="0.02"/>
+                    <!-- <mesh filename="package://little_pig_description/meshes/little_pig_wheel.stl" scale="0.0254 0.0254 0.0254"/> -->
                 </geometry>
             </collision>
@@ -26,4 +27,14 @@
             <limit effort="1.0" velocity="0.5"/>
         </joint>
+        <transmission name="${prefix}_front_wheel_trans">
+            <type>transmission_interface/SimpleTransmission</type>
+            <joint name="${prefix}_front_wheel_joint">
+                <hardwareInterface>hardware_interface/VelocityJointInterface</hardwareInterface>
+            </joint>
+            <actuator name="${prefix}_front_wheel_motor">
+                <hardwareInterface>hardware_interface/VelocityJointInterface</hardwareInterface>
+                <mechanicalReduction>1</mechanicalReduction>
+            </actuator>
+        </transmission>
     </xacro:macro>
 </robot>

File: xacro/macros/_rear_wheel.urdf.xacro (robot description, xacro)
@@ -8,11 +8,12 @@
                     <mesh filename="package://little_pig_description/meshes/little_pig_wheel.stl" scale="0.0254 0.0254 0.0254"/>
                 </geometry>
-                <origin rpy="0 0.0 ${1.57075 * reflect}" xyz="0 0 0.0"/>
+                <origin rpy="0.0 0.0 ${degrees_90 * reflect}" xyz="0 0 0.0"/>
                 <material name="black"/>
             </visual>
             <collision>
-                <origin xyz="0.0 0.0 0.0" rpy="0.0 0.0 ${1.57075 * reflect}"/>
+                <origin xyz="0.0 0.0 0.0" rpy="${degrees_90 * reflect} 0.0 0.0"/>
                 <geometry>
-                    <mesh filename="package://little_pig_description/meshes/little_pig_wheel.stl" scale="0.0254 0.0254 0.0254"/>
+                    <cylinder radius="${rear_wheel_diameter/2}" length="0.02"/>
+                    <!-- <mesh filename="package://little_pig_description/meshes/little_pig_wheel.stl" scale="0.0254 0.0254 0.0254"/> -->
                 </geometry>
             </collision>
@@ -26,4 +27,16 @@
             <limit effort="1.0" velocity="0.5"/>
         </joint>
+        <transmission name="${prefix}_rear_wheel_trans">
+            <type>transmission_interface/SimpleTransmission</type>
+            <joint name="${prefix}_rear_wheel_joint">
+                <!-- <hardwareInterface>hardware_interface/VelocityJointInterface</hardwareInterface> --> <!-- rolling axle -->
+                <hardwareInterface>hardware_interface/EffortJointInterface</hardwareInterface>
+            </joint>
+            <actuator name="${prefix}_rear_wheel_motor">
+                <!-- <hardwareInterface>hardware_interface/VelocityJointInterface</hardwareInterface> --> <!-- rolling axle -->
+                <hardwareInterface>hardware_interface/EffortJointInterface</hardwareInterface>
+                <mechanicalReduction>1</mechanicalReduction>
+            </actuator>
+        </transmission>
     </xacro:macro>
 </robot>

File: xacro/macros/_steering_macro.urdf.xacro (robot description, xacro)
@@ -25,4 +25,14 @@
             <limit lower="-0.30" upper="0.30" effort="1.0" velocity="0.1"/>
         </joint>
+        <transmission name="${prefix}_steer_link_trans">
+            <type>transmission_interface/SimpleTransmission</type>
+            <joint name="${prefix}_steer_joint">
+                <hardwareInterface>hardware_interface/PositionJointInterface</hardwareInterface>
+            </joint>
+            <actuator name="${prefix}_steer_link_motor">
+                <hardwareInterface>hardware_interface/PositionJointInterface</hardwareInterface>
+                <mechanicalReduction>1</mechanicalReduction>
+            </actuator>
+        </transmission>
     </xacro:macro>
 </robot>

Commit message: Add gps, imu, camera and fix some names

File: urdf/little_pig_base.urdf.xacro (robot description, xacro)
@@ -6,4 +6,5 @@
     <xacro:property name="degrees_90" value="1.57079633"/>
     <xacro:property name="degrees_180" value="3.14159265"/>
+    <!-- Included macros -->
     <xacro:include filename="$(find little_pig_description)/xacro/params/color_properties.xacro"/>
     <xacro:include filename="$(find little_pig_description)/xacro/params/characteristics.xacro"/>
@@ -13,4 +14,6 @@
     <xacro:include filename="$(find little_pig_description)/xacro/macros/_front_laser.urdf.xacro" />
     <xacro:include filename="$(find little_pig_description)/xacro/macros/_back_laser.urdf.xacro" />
+    <xacro:include filename="$(find little_pig_description)/xacro/macros/_imu.urdf.xacro" />
+    <xacro:include filename="$(find little_pig_description)/xacro/macros/_camera.urdf.xacro" />
     <!-- Inertia Generator -->
     <xacro:macro name="default_inertial" params="mass">
@@ -20,6 +23,6 @@
         </inertial>
     </xacro:macro>
-    <link name="base_footprint" />
-    <link name="base_link">
+    <link name="base_link" />
+    <link name="chassis">
         <visual>
             <geometry>
@@ -38,8 +41,9 @@
     </link>
     <joint name="base_joint" type="fixed">
-        <parent link="base_footprint"/>
-        <child link="base_link"/>
+        <parent link="base_link"/>
+        <child link="chassis"/>
         <origin xyz="0.0 0.0 0.0" rpy="0 0 0"/>
     </joint>
+    <!-- Call macros to build components -->
     <xacro:steering_component prefix="left" reflect="1" />
     <xacro:steering_component prefix="right" reflect="-1" />
@@ -50,4 +54,6 @@
     <xacro:front_laser />
     <xacro:back_laser />
+    <xacro:imu />
+    <xacro:camera1 />
     <!-- Gazebo plugin for ROS Control -->
     <gazebo>
@@ -55,4 +61,17 @@
             <robotSimType>gazebo_ros_control/AckermannRobotHWSim</robotSimType>
         </plugin>
+        <plugin name="gps_plugin" filename="libhector_gazebo_ros_gps.so">
+            <alwaysOn>1</alwaysOn>
+            <updateRate>40.0</updateRate>
+            <frameId>base_link</frameId> <!-- Defaults to world? don't put in a "/"-->
+            <bodyName>chassis</bodyName>
+            <topicName>fix</topicName>
+            <velocityTopicName>fix_vel</velocityTopicName>
+            <drift>0.0001 0.0001 0.0001</drift>
+            <referenceLatitude>37.634047</referenceLatitude>
+            <referenceLongitude>-97.269368</referenceLongitude>
+            <referenceHeading>0</referenceHeading>
+            <referenceAltitude>0</referenceAltitude>
+        </plugin>
     </gazebo>
 </robot>

File: xacro/macros/_back_laser.urdf.xacro (robot description, xacro)
@@ -7,5 +7,5 @@
             <axis xyz="0 0 0" />
             <origin xyz="-0.8 0.0 0.5" rpy="0 0 ${degrees_180}"/> <!-- Was reversed in real world -->
-            <parent link="base_link"/>
+            <parent link="chassis"/>
             <child link="laser_link_back"/>
         </joint>

File: xacro/macros/_front_laser.urdf.xacro (robot description, xacro)
@@ -7,5 +7,5 @@
             <axis xyz="0 0 0" />
             <origin xyz="1.05 0.0 0.35" rpy="0 0 0"/> <!-- Was reversed in real world -->
-            <parent link="base_link"/>
+            <parent link="chassis"/>
             <child link="laser_link"/>
         </joint>

File: xacro/macros/_front_wheel.urdf.xacro (robot description, xacro)
@@ -17,4 +17,28 @@
                     <!-- <mesh filename="package://little_pig_description/meshes/little_pig_wheel.stl" scale="0.0254 0.0254 0.0254"/> -->
                 </geometry>
+                <surface>
+                    <friction>
+                        <torsional>
+                            <coefficient>2.0</coefficient>
+                            <surface_radius>.3025</surface_radius>
+                            <use_patch_radius>false</use_patch_radius>
+                            <ode>
+                                <slip>0.0</slip>
+                            </ode>
+                        </torsional>
+                        <ode>
+                            <mu>70000.00</mu>
+                            <mu2>70000.00</mu2>
+                            <fdir1>1.00000 0.00000 0.00000</fdir1>
+                            <slip1>0.00000</slip1>
+                            <slip2>0.00000</slip2>
+                        </ode>
+                    </friction>
+                    <contact>
+                        <ode>
+                            <min_depth>0.4025</min_depth>
+                        </ode>
+                    </contact>
+                </surface>
             </collision>
             <xacro:default_inertial mass="${front_wheel_mass}"/>

File: xacro/macros/_rear_wheel.urdf.xacro (robot description, xacro)
@@ -18,10 +18,25 @@
                 </geometry>
             </collision>
+            <surface>
+                <contact>
+                    <ode>
+                        <min_depth>0.01</min_depth>
+                    </ode>
+                </contact>
+                <friction>
+                    <ode>
+                        <mu>1</mu>
+                        <mu2>1</mu2>
+                        <fdir1>1.0 0 0</fdir1>
+                    </ode>
+                </friction>
+            </surface>
             <xacro:default_inertial mass="${rear_wheel_mass}"/>
         </link>
         <joint name="${prefix}_rear_wheel_joint" type="continuous">
-            <parent link="base_link"/>
+            <parent link="chassis"/>
             <child link="${prefix}_rear_wheel"/>
             <origin xyz="-0.65 ${0.45 * reflect} -0.15" rpy="0.0 0.0 0.0"/>
+            <axis xyz="0.0 0.1 0.0"/>
             <!-- <limit effort="1.0" velocity="0.5"/> -->
         </joint>

File: xacro/macros/_steering_macro.urdf.xacro (robot description, xacro)
@@ -19,5 +19,5 @@
         </link>
         <joint name="${prefix}_steer_joint" type="revolute">
-            <parent link="base_link"/>
+            <parent link="chassis"/>
             <child link="${prefix}_steer_link"/>
             <origin xyz="0.7 ${0.45 * reflect} -0.15" rpy="0.0 0.0 0.0"/>

Commit message: Use parameters for positioning

File: urdf/little_pig_base.urdf.xacro (robot description, xacro)
@@ -12,4 +12,5 @@
     <xacro:include filename="$(find little_pig_description)/xacro/macros/_front_wheel.urdf.xacro" />
     <xacro:include filename="$(find little_pig_description)/xacro/macros/_rear_wheel.urdf.xacro" />
+    <!-- Using two laser files due to namespace issues -->
     <xacro:include filename="$(find little_pig_description)/xacro/macros/_front_laser.urdf.xacro" />
     <xacro:include filename="$(find little_pig_description)/xacro/macros/_back_laser.urdf.xacro" />
@@ -52,8 +53,8 @@
     <xacro:rear_wheel prefix="left" reflect="1" />
     <xacro:rear_wheel prefix="right" reflect="-1" />
-    <xacro:front_laser />
-    <xacro:back_laser />
-    <xacro:imu />
-    <xacro:camera1 />
+    <xacro:front_laser position="${front_laser_position}" rotate="0" />
+    <xacro:back_laser position="${back_laser_position}" rotate="${degrees_180}" />
+    <xacro:imu position="${imu_position}"/>
+    <xacro:camera1 position="${camera_position}"/>
     <!-- Gazebo plugin for ROS Control -->
     <gazebo>

File: xacro/macros/_back_laser.urdf.xacro (robot description, xacro)
@@ -2,9 +2,9 @@
 <robot name="back_laser"
     xmlns:xacro="http://ros.org/wiki/xacro">
-    <xacro:macro name="back_laser">
+    <xacro:macro name="back_laser" params="position rotate">
         <!-- Back Laser link -->
         <joint name="laser_link_joint_back" type="fixed">
             <axis xyz="0 0 0" />
-            <origin xyz="-0.8 0.0 0.5" rpy="0 0 ${degrees_180}"/> <!-- Was reversed in real world -->
+            <origin xyz="${position}" rpy="0 0 ${rotate}"/>
             <parent link="chassis"/>
             <child link="laser_link_back"/>
@@ -40,6 +40,6 @@
                             <samples>360</samples>
                             <resolution>1</resolution>
-                            <min_angle>-1.91986</min_angle>
-                            <max_angle>1.91986</max_angle>
+                            <min_angle>-${degrees_90}</min_angle>
+                            <max_angle>${degrees_90}</max_angle>
                         </horizontal>
                     </scan>

File: xacro/macros/_camera.urdf.xacro (robot description, xacro)
@@ -2,8 +2,8 @@
 <robot name="camera1"
     xmlns:xacro="http://ros.org/wiki/xacro">
-    <xacro:macro name="camera1">
+    <xacro:macro name="camera1" params="position">
         <joint name="camera_link_joint" type="fixed">
             <axis xyz="0 1 0" />
-            <origin xyz="1.05 0.0 0.35" rpy="0 0 0"/>
+            <origin xyz="${position}" rpy="0 0 0"/>
             <!-- <origin xyz="1.05 0.0 0.35" rpy="0 0 0"/> -->
             <parent link="chassis"/>

File: xacro/macros/_front_laser.urdf.xacro (robot description, xacro)
@@ -2,9 +2,9 @@
 <robot name="front_laser"
     xmlns:xacro="http://ros.org/wiki/xacro">
-    <xacro:macro name="front_laser">
+    <xacro:macro name="front_laser" params="position rotate">
         <!-- Laser link -->
         <joint name="laser_link_joint" type="fixed">
             <axis xyz="0 0 0" />
-            <origin xyz="1.05 0.0 0.35" rpy="0 0 0"/> <!-- Was reversed in real world -->
+            <origin xyz="${position}" rpy="0 0 ${rotate}"/>
             <parent link="chassis"/>
             <child link="laser_link"/>
@@ -41,6 +41,6 @@
                             <samples>360</samples>
                             <resolution>1</resolution>
-                            <min_angle>-1.91986</min_angle>
-                            <max_angle>1.91986</max_angle>
+                            <min_angle>-${degrees_90}</min_angle>
+                            <max_angle>${degrees_90}</max_angle>
                         </horizontal>
                     </scan>

File: xacro/macros/_imu.urdf.xacro (robot description, xacro)
@@ -2,8 +2,8 @@
 <robot name="imu"
     xmlns:xacro="http://ros.org/wiki/xacro">
-    <xacro:macro name="imu">
+    <xacro:macro name="imu" params="position">
         <joint name="imu_joint" type="fixed">
             <axis xyz="1 0 0 "/> <!-- 0 1 0 -->
-            <origin xyz="0 0 0.19"/>
+            <origin xyz="${position}"/>
             <parent link ="chassis"/>
             <child link ="imu_link"/>

File: xacro/params/characteristics.xacro (robot description, xacro)
@@ -27,3 +27,8 @@
     <xacro:property name="steering_min_angle" value="-${degrees_30}"/>
     <xacro:property name="traverse_max_speed" value="4.785"/> <!-- units of m/s 4.785-->
+    <!-- Module Properties (Positions relative to chassis) -->
+    <xacro:property name="front_laser_position" value="1.05 0.0 0.35" />
+    <xacro:property name="back_laser_position" value="-0.8 0.0 0.5" />
+    <xacro:property name="imu_position" value="0 0 0.19"/>
+    <xacro:property name="camera_position" value="1.05 0.0 0.35"/>
 </robot>
