Commit message: Steering and control fixes

File: xacro/macros/_front_wheel.urdf.xacro (robot description, xacro)
@@ -14,5 +14,5 @@
                 <origin xyz="0.0 0.0 0.0" rpy="${degrees_90 * reflect} 0.0 0.0"/>
                 <geometry>
-                    <cylinder radius="${front_wheel_diameter/2}" length="0.02"/>
+                    <cylinder radius="${front_wheel_diameter/2}" length="${front_wheel_width}"/>
                     <!-- <mesh filename="package://little_pig_description/meshes/little_pig_wheel.stl" scale="0.0254 0.0254 0.0254"/> -->
                 </geometry>
@@ -25,5 +25,6 @@
             <origin xyz="0.0 0.0 0.0" rpy="0.0 0.0 0.0"/>
             <axis xyz="0.0 0.1 0.0"/>
-            <limit effort="1.0" velocity="0.5"/>
+            <!-- <limit effort="1.0" velocity="0.5"/> -->
+            <limit effort="30.00" velocity="${traverse_max_speed * 2 / front_wheel_diameter}"/> <!-- units of rad/s -->
         </joint>
         <transmission name="${prefix}_front_wheel_trans">

File: xacro/macros/_rear_wheel.urdf.xacro (robot description, xacro)
@@ -14,5 +14,5 @@
                 <origin xyz="0.0 0.0 0.0" rpy="${degrees_90 * reflect} 0.0 0.0"/>
                 <geometry>
-                    <cylinder radius="${rear_wheel_diameter/2}" length="0.02"/>
+                    <cylinder radius="${rear_wheel_diameter/2}" length="${rear_wheel_width}"/>
                     <!-- <mesh filename="package://little_pig_description/meshes/little_pig_wheel.stl" scale="0.0254 0.0254 0.0254"/> -->
                 </geometry>
@@ -24,6 +24,5 @@
             <child link="${prefix}_rear_wheel"/>
             <origin xyz="-0.65 ${0.45 * reflect} -0.15" rpy="0.0 0.0 0.0"/>
-            <axis xyz="0.0 0.1 0.0"/>
-            <limit effort="1.0" velocity="0.5"/>
+            <!-- <limit effort="1.0" velocity="0.5"/> -->
         </joint>
         <transmission name="${prefix}_rear_wheel_trans">

File: xacro/macros/_steering_macro.urdf.xacro (robot description, xacro)
@@ -23,5 +23,6 @@
             <origin xyz="0.7 ${0.45 * reflect} -0.15" rpy="0.0 0.0 0.0"/>
             <axis xyz="0.0 0.0 0.1"/>
-            <limit lower="-0.30" upper="0.30" effort="1.0" velocity="0.1"/>
+            <limit lower="${steering_min_angle}" upper="${steering_max_angle}" effort="30.00" velocity="${steering_speed}"/>
+            <!-- <limit lower="-0.30" upper="0.30" effort="1.0" velocity="0.1"/> -->
         </joint>
         <transmission name="${prefix}_steer_link_trans">

File: xacro/params/characteristics.xacro (robot description, xacro)
@@ -11,18 +11,19 @@
     <xacro:property name="front_wheel_diameter" value="0.572" />
     <xacro:property name="front_wheel_mass" value="20"/>
+    <!-- Steering Link Properties -->
+    <xacro:property name="steering_width" value="${front_wheel_width/4}" />
+    <xacro:property name="steering_diameter" value="${front_wheel_diameter/5}" />
+    <xacro:property name="steering_mass" value="2"/>
     <!-- Rear Wheel Properties -->
     <xacro:property name="rear_wheel_width" value="${front_wheel_width+steering_width}" />
     <xacro:property name="rear_wheel_diameter" value="0.635" />
     <xacro:property name="rear_wheel_mass" value="22.8"/>
-    <!-- Steering Link Properties -->
-    <xacro:property name="steering_width" value="${front_wheel_width/4}" />
-    <xacro:property name="steering_diameter" value="${front_wheel_diameter/5}" />
-    <xacro:property name="steering_mass" value="2"/>
     <!-- Steering Characteristics -->
     <!-- units of rad/s -->
     <xacro:property name="steering_speed" value="1.0472"/>
     <!-- units of rad, used to be 0.523 -->
-    <xacro:property name="steering_max_angle" value="${degrees_45}"/>
+    <xacro:property name="steering_max_angle" value="${degrees_30}"/>
     <!-- units of rad, used to be 0.523 -->
-    <xacro:property name="steering_min_angle" value="-${degrees_45}"/>
+    <xacro:property name="steering_min_angle" value="-${degrees_30}"/>
+    <xacro:property name="traverse_max_speed" value="4.785"/> <!-- units of m/s 4.785-->
 </robot>
