Commit message: Updating specifications of simulation lasers

File: xacro/macros/_back_laser.urdf.xacro (robot description, xacro)
@@ -38,5 +38,5 @@
                     <scan>
                         <horizontal>
-                            <samples>360</samples>
+                            <samples>460</samples>
                             <resolution>1</resolution>
                             <min_angle>-${degrees_90}</min_angle>
@@ -47,5 +47,5 @@
                         <min>0.10</min>
                         <max>20.0</max>
-                        <resolution>0.05</resolution>
+                        <resolution>0.03</resolution>
                     </range>
                     <noise>

File: xacro/macros/_front_laser.urdf.xacro (robot description, xacro)
@@ -15,5 +15,5 @@
                 <origin xyz="0 0 0" rpy="0 0 0"/>
                 <geometry>
-                    <cylinder radius=".05" length="0.04"/>
+                    <cylinder radius=".055" length="0.051"/>
                 </geometry>
             </collision>
@@ -21,5 +21,5 @@
                 <origin xyz="0 0 0" rpy="0 0 0"/>
                 <geometry>
-                    <cylinder radius=".05" length="0.04"/>
+                    <cylinder radius=".055" length="0.051"/>
                 </geometry>
             </visual>
@@ -39,5 +39,5 @@
                     <scan>
                         <horizontal>
-                            <samples>360</samples>
+                            <samples>460</samples>
                             <resolution>1</resolution>
                             <min_angle>-${degrees_90}</min_angle>
@@ -48,5 +48,5 @@
                         <min>0.10</min>
                         <max>20.0</max>
-                        <resolution>0.05</resolution>
+                        <resolution>0.03</resolution>
                     </range>
                     <noise>

File: xacro/params/characteristics.xacro (robot description, xacro)
@@ -28,6 +28,6 @@
     <xacro:property name="traverse_max_speed" value="4.785"/> <!-- units of m/s 4.785-->
     <!-- Module Properties (Positions relative to chassis) -->
-    <xacro:property name="front_laser_position" value="1.05 0.0 0.35" />
-    <xacro:property name="back_laser_position" value="-0.8 0.0 0.5" />
+    <xacro:property name="front_laser_position" value="1.05 0.0 0.038" />
+    <xacro:property name="back_laser_position" value="-0.8 0.0 0.13" />
     <xacro:property name="imu_position" value="0 0 0.19"/>
     <xacro:property name="camera_position" value="1.05 0.0 0.35"/>

Commit message: Updating specifications of simulation lasers

File: xacro/macros/_back_laser.urdf.xacro (robot description, xacro)
@@ -14,5 +14,5 @@
                 <origin xyz="0 0 0" rpy="0 0 0"/>
                 <geometry>
-                    <cylinder radius=".05" length="0.04"/>
+                    <cylinder radius=".055" length="0.051"/>
                 </geometry>
             </collision>
@@ -20,5 +20,5 @@
                 <origin xyz="0 0 0" rpy="0 0 0"/>
                 <geometry>
-                    <cylinder radius=".05" length="0.04"/>
+                    <cylinder radius=".055" length="0.051"/>
                 </geometry>
             </visual>
@@ -47,5 +47,5 @@
                         <min>0.10</min>
                         <max>20.0</max>
-                        <resolution>0.03</resolution>
+                        <resolution>0.03</resolution> <!-- Distance Resolution -->
                     </range>
                     <noise>

File: xacro/macros/_front_laser.urdf.xacro (robot description, xacro)
@@ -48,5 +48,5 @@
                         <min>0.10</min>
                         <max>20.0</max>
-                        <resolution>0.03</resolution>
+                        <resolution>0.03</resolution> <!-- Distance Resolution -->
                     </range>
                     <noise>

File: xacro/params/characteristics.xacro (robot description, xacro)
@@ -29,5 +29,5 @@
     <!-- Module Properties (Positions relative to chassis) -->
     <xacro:property name="front_laser_position" value="1.05 0.0 0.038" />
-    <xacro:property name="back_laser_position" value="-0.8 0.0 0.13" />
+    <xacro:property name="back_laser_position" value="-0.8 0.0 0.13" /> <!-- Height needs to be adjusted once we see real-world Little Pig-->
     <xacro:property name="imu_position" value="0 0 0.19"/>
     <xacro:property name="camera_position" value="1.05 0.0 0.35"/>
